Commit message: Added rh_5_left URDF
Signed-off-by: Hyunwoo Nam <nhw@robotis.com>

File: robotis_hand_description/urdf/rh_5_right.urdf.xacro (robot description, xacro)
@@ -2,5 +2,5 @@
 <robot xmlns:xacro="http://www.ros.org/wiki/xacro" name="robotis_hand">
    <xacro:macro name="robotis_hand" params="prefix">
-      <xacro:property name="meshes_file_direction" value="package://robotis_hand_description/meshes/" />
+      <xacro:property name="meshes_file_direction" value="package://robotis_hand_description/meshes/rh_5_right/" />
       <link name="${prefix}robotis_hand_base">
          <visual>

File: robotis_hand_description/urdf/rh_5_right.xacro (robot description, xacro)
@@ -5,6 +5,6 @@
   <xacro:arg name="use_fake_hardware" default="false" />
   <xacro:arg name="fake_sensor_commands" default="false" />
-  <xacro:include filename="$(find robotis_hand_description)/urdf/robotis_hand.xacro" />
-  <xacro:include filename="$(find robotis_hand_description)/gazebo/rh_5_right.gazebo.xacro" />
+  <xacro:include filename="$(find robotis_hand_description)/urdf/rh_5_right.urdf.xacro" />
+  <xacro:include filename="$(find robotis_hand_description)/gazebo/robotis_hand.gazebo.xacro" />
   <xacro:include filename="$(find robotis_hand_description)/ros2_control/robotis_hand.ros2_control.xacro" />
   <link name="world"/>
