Commit message: Updated ROS 2 packages for ros2_control
Signed-off-by: Hyunwoo Nam <nhw@robotis.com>

File: robotis_hand_description/ros2_control/robotis_hand.ros2_control.xacro (robot description, xacro)
@@ -21,12 +21,50 @@
             <param name="error_timeout_ms">500</param>
             <param name="dynamixel_model_folder">/param/dxl_model</param>
-            <param name="number_of_joints">1</param>
-            <param name="number_of_transmissions">1</param>
+            <param name="number_of_joints">20</param>
+            <param name="number_of_transmissions">20</param>
             <param name="disable_torque_at_init">true</param>
             <param name="transmission_to_joint_matrix">
-              1
+              1, 0, 0, 0, 0, 0, 0, 0, 0, 0, 0, 0, 0, 0, 0, 0, 0, 0, 0, 0,
+              0, 1, 0, 0, 0, 0, 0, 0, 0, 0, 0, 0, 0, 0, 0, 0, 0, 0, 0, 0,
+              0, 0, 1, 0, 0, 0, 0, 0, 0, 0, 0, 0, 0, 0, 0, 0, 0, 0, 0, 0,
+              0, 0, 0, 1, 0, 0, 0, 0, 0, 0, 0, 0, 0, 0, 0, 0, 0, 0, 0, 0,
+              0, 0, 0, 0, 1, 0, 0, 0, 0, 0, 0, 0, 0, 0, 0, 0, 0, 0, 0, 0,
+              0, 0, 0, 0, 0, 1, 0, 0, 0, 0, 0, 0, 0, 0, 0, 0, 0, 0, 0, 0,
+              0, 0, 0, 0, 0, 0, 1, 0, 0, 0, 0, 0, 0, 0, 0, 0, 0, 0, 0, 0,
+              0, 0, 0, 0, 0, 0, 0, 1, 0, 0, 0, 0, 0, 0, 0, 0, 0, 0, 0, 0,
+              0, 0, 0, 0, 0, 0, 0, 0, 1, 0, 0, 0, 0, 0, 0, 0, 0, 0, 0, 0,
+              0, 0, 0, 0, 0, 0, 0, 0, 0, 1, 0, 0, 0, 0, 0, 0, 0, 0, 0, 0,
+              0, 0, 0, 0, 0, 0, 0, 0, 0, 0, 1, 0, 0, 0, 0, 0, 0, 0, 0, 0,
+              0, 0, 0, 0, 0, 0, 0, 0, 0, 0, 0, 1, 0, 0, 0, 0, 0, 0, 0, 0,
+              0, 0, 0, 0, 0, 0, 0, 0, 0, 0, 0, 0, 1, 0, 0, 0, 0, 0, 0, 0,
+              0, 0, 0, 0, 0, 0, 0, 0, 0, 0, 0, 0, 0, 1, 0, 0, 0, 0, 0, 0,
+              0, 0, 0, 0, 0, 0, 0, 0, 0, 0, 0, 0, 0, 0, 1, 0, 0, 0, 0, 0,
+              0, 0, 0, 0, 0, 0, 0, 0, 0, 0, 0, 0, 0, 0, 0, 1, 0, 0, 0, 0,
+              0, 0, 0, 0, 0, 0, 0, 0, 0, 0, 0, 0, 0, 0, 0, 0, 1, 0, 0, 0,
+              0, 0, 0, 0, 0, 0, 0, 0, 0, 0, 0, 0, 0, 0, 0, 0, 0, 1, 0, 0,
+              0, 0, 0, 0, 0, 0, 0, 0, 0, 0, 0, 0, 0, 0, 0, 0, 0, 0, 1, 0,
+              0, 0, 0, 0, 0, 0, 0, 0, 0, 0, 0, 0, 0, 0, 0, 0, 0, 0, 0, 1
             </param>
             <param name="joint_to_transmission_matrix">
-              1
+              1, 0, 0, 0, 0, 0, 0, 0, 0, 0, 0, 0, 0, 0, 0, 0, 0, 0, 0, 0,
+              0, 1, 0, 0, 0, 0, 0, 0, 0, 0, 0, 0, 0, 0, 0, 0, 0, 0, 0, 0,
+              0, 0, 1, 0, 0, 0, 0, 0, 0, 0, 0, 0, 0, 0, 0, 0, 0, 0, 0, 0,
+              0, 0, 0, 1, 0, 0, 0, 0, 0, 0, 0, 0, 0, 0, 0, 0, 0, 0, 0, 0,
+              0, 0, 0, 0, 1, 0, 0, 0, 0, 0, 0, 0, 0, 0, 0, 0, 0, 0, 0, 0,
+              0, 0, 0, 0, 0, 1, 0, 0, 0, 0, 0, 0, 0, 0, 0, 0, 0, 0, 0, 0,
+              0, 0, 0, 0, 0, 0, 1, 0, 0, 0, 0, 0, 0, 0, 0, 0, 0, 0, 0, 0,
+              0, 0, 0, 0, 0, 0, 0, 1, 0, 0, 0, 0, 0, 0, 0, 0, 0, 0, 0, 0,
+              0, 0, 0, 0, 0, 0, 0, 0, 1, 0, 0, 0, 0, 0, 0, 0, 0, 0, 0, 0,
+              0, 0, 0, 0, 0, 0, 0, 0, 0, 1, 0, 0, 0, 0, 0, 0, 0, 0, 0, 0,
+              0, 0, 0, 0, 0, 0, 0, 0, 0, 0, 1, 0, 0, 0, 0, 0, 0, 0, 0, 0,
+              0, 0, 0, 0, 0, 0, 0, 0, 0, 0, 0, 1, 0, 0, 0, 0, 0, 0, 0, 0,
+              0, 0, 0, 0, 0, 0, 0, 0, 0, 0, 0, 0, 1, 0, 0, 0, 0, 0, 0, 0,
+              0, 0, 0, 0, 0, 0, 0, 0, 0, 0, 0, 0, 0, 1, 0, 0, 0, 0, 0, 0,
+              0, 0, 0, 0, 0, 0, 0, 0, 0, 0, 0, 0, 0, 0, 1, 0, 0, 0, 0, 0,
+              0, 0, 0, 0, 0, 0, 0, 0, 0, 0, 0, 0, 0, 0, 0, 1, 0, 0, 0, 0,
+              0, 0, 0, 0, 0, 0, 0, 0, 0, 0, 0, 0, 0, 0, 0, 0, 1, 0, 0, 0,
+              0, 0, 0, 0, 0, 0, 0, 0, 0, 0, 0, 0, 0, 0, 0, 0, 0, 1, 0, 0,
+              0, 0, 0, 0, 0, 0, 0, 0, 0, 0, 0, 0, 0, 0, 0, 0, 0, 0, 1, 0,
+              0, 0, 0, 0, 0, 0, 0, 0, 0, 0, 0, 0, 0, 0, 0, 0, 0, 0, 0, 1
             </param>
             <param name="dynamixel_state_pub_msg_name">dynamixel_hardware_interface/dxl_state</param>
@@ -38,39 +76,124 @@
         </hardware>
       </xacro:unless>
-      <joint name="${prefix}rh_r1">
-        <command_interface name="position"/>
-        <state_interface name="position"/>
-        <state_interface name="velocity"/>
-        <state_interface name="effort"/>
-      </joint>
-      <xacro:if value="$(arg use_sim)">
-        <joint name="${prefix}rh_r2">
-          <param name="mimic">${prefix}rh_r1</param>
-          <param name="multiplier">1</param>
-          <state_interface name="position"/>
-          <state_interface name="velocity"/>
-          <state_interface name="effort"/>
-          <state_interface name="torque_enable"/>
-          <state_interface name="hardware_state"/>
-        </joint>
-        <joint name="${prefix}rh_l1">
-          <param name="mimic">${prefix}rh_r1</param>
-          <param name="multiplier">1</param>
-          <state_interface name="position"/>
-          <state_interface name="velocity"/>
-          <state_interface name="effort"/>
-          <state_interface name="torque_enable"/>
-          <state_interface name="hardware_state"/>
-        </joint>
-        <joint name="${prefix}rh_l2">
-          <param name="mimic">${prefix}rh_r1</param>
-          <param name="multiplier">1</param>
-          <state_interface name="position"/>
-          <state_interface name="velocity"/>
-          <state_interface name="effort"/>
-          <state_interface name="torque_enable"/>
-          <state_interface name="hardware_state"/>
-        </joint>
-      </xacro:if>
+      <joint name="${prefix}finger_joint_1">
+        <command_interface name="position"/>
+        <state_interface name="position"/>
+        <state_interface name="velocity"/>
+        <state_interface name="effort"/>
+      </joint>
+      <joint name="${prefix}finger_joint_2">
+        <command_interface name="position"/>
+        <state_interface name="position"/>
+        <state_interface name="velocity"/>
+        <state_interface name="effort"/>
+      </joint>
+      <joint name="${prefix}finger_joint_3">
+        <command_interface name="position"/>
+        <state_interface name="position"/>
+        <state_interface name="velocity"/>
+        <state_interface name="effort"/>
+      </joint>
+      <joint name="${prefix}finger_joint_4">
+        <command_interface name="position"/>
+        <state_interface name="position"/>
+        <state_interface name="velocity"/>
+        <state_interface name="effort"/>
+      </joint>
+      <joint name="${prefix}finger_joint_5">
+        <command_interface name="position"/>
+        <state_interface name="position"/>
+        <state_interface name="velocity"/>
+        <state_interface name="effort"/>
+      </joint>
+      <joint name="${prefix}finger_joint_6">
+        <command_interface name="position"/>
+        <state_interface name="position"/>
+        <state_interface name="velocity"/>
+        <state_interface name="effort"/>
+      </joint>
+      <joint name="${prefix}finger_joint_7">
+        <command_interface name="position"/>
+        <state_interface name="position"/>
+        <state_interface name="velocity"/>
+        <state_interface name="effort"/>
+      </joint>
+      <joint name="${prefix}finger_joint_8">
+        <command_interface name="position"/>
+        <state_interface name="position"/>
+        <state_interface name="velocity"/>
+        <state_interface name="effort"/>
+      </joint>
+      <joint name="${prefix}finger_joint_9">
+        <command_interface name="position"/>
+        <state_interface name="position"/>
+        <state_interface name="velocity"/>
+        <state_interface name="effort"/>
+      </joint>
+      <joint name="${prefix}finger_joint_10">
+        <command_interface name="position"/>
+        <state_interface name="position"/>
+        <state_interface name="velocity"/>
+        <state_interface name="effort"/>
+      </joint>
+      <joint name="${prefix}finger_joint_11">
+        <command_interface name="position"/>
+        <state_interface name="position"/>
+        <state_interface name="velocity"/>
+        <state_interface name="effort"/>
+      </joint>
+      <joint name="${prefix}finger_joint_12">
+        <command_interface name="position"/>
+        <state_interface name="position"/>
+        <state_interface name="velocity"/>
+        <state_interface name="effort"/>
+      </joint>
+      <joint name="${prefix}finger_joint_13">
+        <command_interface name="position"/>
+        <state_interface name="position"/>
+        <state_interface name="velocity"/>
+        <state_interface name="effort"/>
+      </joint>
+      <joint name="${prefix}finger_joint_14">
+        <command_interface name="position"/>
+        <state_interface name="position"/>
+        <state_interface name="velocity"/>
+        <state_interface name="effort"/>
+      </joint>
+      <joint name="${prefix}finger_joint_15">
+        <command_interface name="position"/>
+        <state_interface name="position"/>
+        <state_interface name="velocity"/>
+        <state_interface name="effort"/>
+      </joint>
+      <joint name="${prefix}finger_joint_16">
+        <command_interface name="position"/>
+        <state_interface name="position"/>
+        <state_interface name="velocity"/>
+        <state_interface name="effort"/>
+      </joint>
+      <joint name="${prefix}finger_joint_17">
+        <command_interface name="position"/>
+        <state_interface name="position"/>
+        <state_interface name="velocity"/>
+        <state_interface name="effort"/>
+      </joint>
+      <joint name="${prefix}finger_joint_18">
+        <command_interface name="position"/>
+        <state_interface name="position"/>
+        <state_interface name="velocity"/>
+        <state_interface name="effort"/>
+      </joint>
+      <joint name="${prefix}finger_joint_19">
+        <command_interface name="position"/>
+        <state_interface name="position"/>
+        <state_interface name="velocity"/>
+        <state_interface name="effort"/>
+      </joint>
+      <joint name="${prefix}finger_joint_20">
+        <command_interface name="position"/>
+        <state_interface name="position"/>
+        <state_interface name="velocity"/>
+        <state_interface name="effort"/>
+      </joint>
       <gpio name="dxl1">
         <command_interface name="Goal Position"/>
@@ -82,5 +205,252 @@
         <param name="Return Delay Time">0</param>
         <param name="Min Position Limit">0</param>
-        <param name="Max Position Limit">740</param>
+        <param name="Max Position Limit">4095</param>
+        <param name="Profile Acceleration">0</param>
+        <param name="Profile Velocity">0</param>
+      </gpio>
+      <gpio name="dxl2">
+        <command_interface name="Goal Position"/>
+        <state_interface name="Present Position"/>
+        <state_interface name="Present Velocity"/>
+        <state_interface name="Present Current"/>
+        <param name="type">dxl</param>
+        <param name="ID">2</param>
+        <param name="Return Delay Time">0</param>
+        <param name="Min Position Limit">0</param>
+        <param name="Max Position Limit">4095</param>
+        <param name="Profile Acceleration">0</param>
+        <param name="Profile Velocity">0</param>
+      </gpio>
+      <gpio name="dxl3">
+        <command_interface name="Goal Position"/>
+        <state_interface name="Present Position"/>
+        <state_interface name="Present Velocity"/>
+        <state_interface name="Present Current"/>
+        <param name="type">dxl</param>
+        <param name="ID">3</param>
+        <param name="Return Delay Time">0</param>
+        <param name="Min Position Limit">0</param>
+        <param name="Max Position Limit">4095</param>
+        <param name="Profile Acceleration">0</param>
+        <param name="Profile Velocity">0</param>
+      </gpio>
+      <gpio name="dxl4">
+        <command_interface name="Goal Position"/>
+        <state_interface name="Present Position"/>
+        <state_interface name="Present Velocity"/>
+        <state_interface name="Present Current"/>
+        <param name="type">dxl</param>
+        <param name="ID">4</param>
+        <param name="Return Delay Time">0</param>
+        <param name="Min Position Limit">0</param>
+        <param name="Max Position Limit">4095</param>
+        <param name="Profile Acceleration">0</param>
+        <param name="Profile Velocity">0</param>
+      </gpio>
+      <gpio name="dxl5">
+        <command_interface name="Goal Position"/>
+        <state_interface name="Present Position"/>
+        <state_interface name="Present Velocity"/>
+        <state_interface name="Present Current"/>
+        <param name="type">dxl</param>
+        <param name="ID">5</param>
+        <param name="Return Delay Time">0</param>
+        <param name="Min Position Limit">0</param>
+        <param name="Max Position Limit">4095</param>
+        <param name="Profile Acceleration">0</param>
+        <param name="Profile Velocity">0</param>
+      </gpio>
+      <gpio name="dxl6">
+        <command_interface name="Goal Position"/>
+        <state_interface name="Present Position"/>
+        <state_interface name="Present Velocity"/>
+        <state_interface name="Present Current"/>
+        <param name="type">dxl</param>
+        <param name="ID">6</param>
+        <param name="Return Delay Time">0</param>
+        <param name="Min Position Limit">0</param>
+        <param name="Max Position Limit">4095</param>
+        <param name="Profile Acceleration">0</param>
+        <param name="Profile Velocity">0</param>
+      </gpio>
+      <gpio name="dxl7">
+        <command_interface name="Goal Position"/>
+        <state_interface name="Present Position"/>
+        <state_interface name="Present Velocity"/>
+        <state_interface name="Present Current"/>
+        <param name="type">dxl</param>
+        <param name="ID">7</param>
+        <param name="Return Delay Time">0</param>
+        <param name="Min Position Limit">0</param>
+        <param name="Max Position Limit">4095</param>
+        <param name="Profile Acceleration">0</param>
+        <param name="Profile Velocity">0</param>
+      </gpio>
+      <gpio name="dxl8">
+        <command_interface name="Goal Position"/>
+        <state_interface name="Present Position"/>
+        <state_interface name="Present Velocity"/>
+        <state_interface name="Present Current"/>
+        <param name="type">dxl</param>
+        <param name="ID">8</param>
+        <param name="Return Delay Time">0</param>
+        <param name="Min Position Limit">0</param>
+        <param name="Max Position Limit">4095</param>
+        <param name="Profile Acceleration">0</param>
+        <param name="Profile Velocity">0</param>
+      </gpio>
+      <gpio name="dxl9">
+        <command_interface name="Goal Position"/>
+        <state_interface name="Present Position"/>
+        <state_interface name="Present Velocity"/>
+        <state_interface name="Present Current"/>
+        <param name="type">dxl</param>
+        <param name="ID">9</param>
+        <param name="Return Delay Time">0</param>
+        <param name="Min Position Limit">0</param>
+        <param name="Max Position Limit">4095</param>
+        <param name="Profile Acceleration">0</param>
+        <param name="Profile Velocity">0</param>
+      </gpio>
+      <gpio name="dxl10">
+        <command_interface name="Goal Position"/>
+        <state_interface name="Present Position"/>
+        <state_interface name="Present Velocity"/>
+        <state_interface name="Present Current"/>
+        <param name="type">dxl</param>
+        <param name="ID">10</param>
+        <param name="Return Delay Time">0</param>
+        <param name="Min Position Limit">0</param>
+        <param name="Max Position Limit">4095</param>
+        <param name="Profile Acceleration">0</param>
+        <param name="Profile Velocity">0</param>
+      </gpio>
+      <gpio name="dxl11">
+        <command_interface name="Goal Position"/>
+        <state_interface name="Present Position"/>
+        <state_interface name="Present Velocity"/>
+        <state_interface name="Present Current"/>
+        <param name="type">dxl</param>
+        <param name="ID">11</param>
+        <param name="Return Delay Time">0</param>
+        <param name="Min Position Limit">0</param>
+        <param name="Max Position Limit">4095</param>
+        <param name="Profile Acceleration">0</param>
+        <param name="Profile Velocity">0</param>
+      </gpio>
+      <gpio name="dxl12">
+        <command_interface name="Goal Position"/>
+        <state_interface name="Present Position"/>
+        <state_interface name="Present Velocity"/>
+        <state_interface name="Present Current"/>
+        <param name="type">dxl</param>
+        <param name="ID">12</param>
+        <param name="Return Delay Time">0</param>
+        <param name="Min Position Limit">0</param>
+        <param name="Max Position Limit">4095</param>
+        <param name="Profile Acceleration">0</param>
+        <param name="Profile Velocity">0</param>
+      </gpio>
+      <gpio name="dxl13">
+        <command_interface name="Goal Position"/>
+        <state_interface name="Present Position"/>
+        <state_interface name="Present Velocity"/>
+        <state_interface name="Present Current"/>
+        <param name="type">dxl</param>
+        <param name="ID">13</param>
+        <param name="Return Delay Time">0</param>
+        <param name="Min Position Limit">0</param>
+        <param name="Max Position Limit">4095</param>
+        <param name="Profile Acceleration">0</param>
+        <param name="Profile Velocity">0</param>
+      </gpio>
+      <gpio name="dxl14">
+        <command_interface name="Goal Position"/>
+        <state_interface name="Present Position"/>
+        <state_interface name="Present Velocity"/>
+        <state_interface name="Present Current"/>
+        <param name="type">dxl</param>
+        <param name="ID">14</param>
+        <param name="Return Delay Time">0</param>
+        <param name="Min Position Limit">0</param>
+        <param name="Max Position Limit">4095</param>
+        <param name="Profile Acceleration">0</param>
+        <param name="Profile Velocity">0</param>
+      </gpio>
+      <gpio name="dxl15">
+        <command_interface name="Goal Position"/>
+        <state_interface name="Present Position"/>
+        <state_interface name="Present Velocity"/>
+        <state_interface name="Present Current"/>
+        <param name="type">dxl</param>
+        <param name="ID">15</param>
+        <param name="Return Delay Time">0</param>
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
File: robotis_hand_description/urdf/robotis_hand.urdf.xacro (robot description, xacro)
@@ -2,10 +2,10 @@
 <robot name="robotis_hand" xmlns:xacro="http://www.ros.org/wiki/xacro">
   <xacro:arg name="prefix" default="" />
-  <!-- <xacro:arg name="use_sim" default="false" />
+  <xacro:arg name="use_sim" default="false" />
   <xacro:arg name="use_fake_hardware" default="false" />
-  <xacro:arg name="fake_sensor_commands" default="false" /> -->
+  <xacro:arg name="fake_sensor_commands" default="false" />
   <xacro:include filename="$(find robotis_hand_description)/urdf/robotis_hand.xacro" />
-  <!-- <xacro:include filename="$(find robotis_hand_description)/gazebo/robotis_hand.gazebo.xacro" /> -->
-  <!-- <xacro:include filename="$(find robotis_hand_description)/ros2_control/robotis_hand.ros2_control.xacro" /> -->
+  <xacro:include filename="$(find robotis_hand_description)/gazebo/rh_5_right.gazebo.xacro" />
+  <xacro:include filename="$(find robotis_hand_description)/ros2_control/robotis_hand.ros2_control.xacro" />
   <link name="world"/>
   <joint name="$(arg prefix)world_fixed" type="fixed">
@@ -15,13 +15,13 @@
   </joint>
   <xacro:robotis_hand prefix="$(arg prefix)" />
-  <!-- <xacro:robotis_hand_gazebo prefix="$(arg prefix)" /> -->
-  <!-- <xacro:robotis_hand_system
+  <xacro:robotis_hand_gazebo prefix="$(arg prefix)" />
+  <xacro:robotis_hand_system
     name="RobotisHandSystem" prefix="$(arg prefix)" use_sim="$(arg use_sim)"
     use_fake_hardware="$(arg use_fake_hardware)"
-    fake_sensor_commands="$(arg fake_sensor_commands)"/> -->
-  <!-- <gazebo>
+    fake_sensor_commands="$(arg fake_sensor_commands)"/>
+  <gazebo>
     <plugin filename="gz_ros2_control-system" name="gz_ros2_control::GazeboSimROS2ControlPlugin">
       <parameters>$(find robotis_hand_bringup)/config/hardware_controller_manager.yaml</parameters>
     </plugin>
-  </gazebo> -->
+  </gazebo>
 </robot>
