Commit message: feat: add ros2_control

File: robotis_hand_description/ros2_control/robotis_hand.ros2_control.xacro (robot description, xacro)
@@ -18,5 +18,5 @@
             <plugin>dynamixel_hardware_interface/DynamixelHardware</plugin>
             <param name="port_name">${port_name}</param>
-            <param name="baud_rate">4000000</param>
+            <param name="baud_rate">6000000</param>
             <param name="error_timeout_ms">500</param>
             <param name="dynamixel_model_folder">/param/dxl_model</param>
@@ -78,4 +78,5 @@
       <joint name="${prefix}finger_joint_1">
         <command_interface name="position"/>
+        <command_interface name="effort"/>
         <state_interface name="position"/>
         <state_interface name="velocity"/>
@@ -84,4 +85,5 @@
       <joint name="${prefix}finger_joint_2">
         <command_interface name="position"/>
+        <command_interface name="effort"/>
         <state_interface name="position"/>
         <state_interface name="velocity"/>
@@ -90,4 +92,5 @@
       <joint name="${prefix}finger_joint_3">
         <command_interface name="position"/>
+        <command_interface name="effort"/>
         <state_interface name="position"/>
         <state_interface name="velocity"/>
@@ -96,10 +99,23 @@
       <joint name="${prefix}finger_joint_4">
         <command_interface name="position"/>
-        <state_interface name="position"/>
-        <state_interface name="velocity"/>
-        <state_interface name="effort"/>
-      </joint>
+        <command_interface name="effort"/>
+        <state_interface name="position"/>
+        <state_interface name="velocity"/>
+        <state_interface name="effort"/>
+      </joint>
+      <sensor name="${prefix}finger_sensor_1">
+        <state_interface name="Present Pressure 1"/>
+        <state_interface name="Present Pressure 2"/>
+        <state_interface name="Present Pressure 3"/>
+        <state_interface name="Present Pressure 4"/>
+        <state_interface name="Present Pressure 5"/>
+        <state_interface name="Present Pressure 6"/>
+        <state_interface name="Present Pressure 7"/>
+        <state_interface name="Present Pressure 8"/>
+        <state_interface name="Present Pressure 9"/>
+      </sensor>
       <joint name="${prefix}finger_joint_5">
         <command_interface name="position"/>
+        <command_interface name="effort"/>
         <state_interface name="position"/>
         <state_interface name="velocity"/>
@@ -108,4 +124,5 @@
       <joint name="${prefix}finger_joint_6">
         <command_interface name="position"/>
+        <command_interface name="effort"/>
         <state_interface name="position"/>
         <state_interface name="velocity"/>
@@ -114,4 +131,5 @@
       <joint name="${prefix}finger_joint_7">
         <command_interface name="position"/>
+        <command_interface name="effort"/>
         <state_interface name="position"/>
         <state_interface name="velocity"/>
@@ -120,10 +138,23 @@
       <joint name="${prefix}finger_joint_8">
         <command_interface name="position"/>
-        <state_interface name="position"/>
-        <state_interface name="velocity"/>
-        <state_interface name="effort"/>
-      </joint>
+        <command_interface name="effort"/>
+        <state_interface name="position"/>
+        <state_interface name="velocity"/>
+        <state_interface name="effort"/>
+      </joint>
+      <sensor name="${prefix}finger_sensor_2">
+        <state_interface name="Present Pressure 1"/>
+        <state_interface name="Present Pressure 2"/>
+        <state_interface name="Present Pressure 3"/>
+        <state_interface name="Present Pressure 4"/>
+        <state_interface name="Present Pressure 5"/>
+        <state_interface name="Present Pressure 6"/>
+        <state_interface name="Present Pressure 7"/>
+        <state_interface name="Present Pressure 8"/>
+        <state_interface name="Present Pressure 9"/>
+      </sensor>
       <joint name="${prefix}finger_joint_9">
         <command_interface name="position"/>
+        <command_interface name="effort"/>
         <state_interface name="position"/>
         <state_interface name="velocity"/>
@@ -132,4 +163,5 @@
       <joint name="${prefix}finger_joint_10">
         <command_interface name="position"/>
+        <command_interface name="effort"/>
         <state_interface name="position"/>
         <state_interface name="velocity"/>
@@ -138,4 +170,5 @@
       <joint name="${prefix}finger_joint_11">
         <command_interface name="position"/>
+        <command_interface name="effort"/>
         <state_interface name="position"/>
         <state_interface name="velocity"/>
@@ -144,10 +177,23 @@
       <joint name="${prefix}finger_joint_12">
         <command_interface name="position"/>
-        <state_interface name="position"/>
-        <state_interface name="velocity"/>
-        <state_interface name="effort"/>
-      </joint>
+        <command_interface name="effort"/>
+        <state_interface name="position"/>
+        <state_interface name="velocity"/>
+        <state_interface name="effort"/>
+      </joint>
+      <sensor name="${prefix}finger_sensor_3">
+        <state_interface name="Present Pressure 1"/>
+        <state_interface name="Present Pressure 2"/>
+        <state_interface name="Present Pressure 3"/>
+        <state_interface name="Present Pressure 4"/>
+        <state_interface name="Present Pressure 5"/>
+        <state_interface name="Present Pressure 6"/>
+        <state_interface name="Present Pressure 7"/>
+        <state_interface name="Present Pressure 8"/>
+        <state_interface name="Present Pressure 9"/>
+      </sensor>
       <joint name="${prefix}finger_joint_13">
         <command_interface name="position"/>
+        <command_interface name="effort"/>
         <state_interface name="position"/>
         <state_interface name="velocity"/>
@@ -156,4 +202,5 @@
       <joint name="${prefix}finger_joint_14">
         <command_interface name="position"/>
+        <command_interface name="effort"/>
         <state_interface name="position"/>
         <state_interface name="velocity"/>
@@ -162,4 +209,5 @@
       <joint name="${prefix}finger_joint_15">
         <command_interface name="position"/>
+        <command_interface name="effort"/>
         <state_interface name="position"/>
         <state_interface name="velocity"/>
@@ -168,10 +216,23 @@
       <joint name="${prefix}finger_joint_16">
         <command_interface name="position"/>
-        <state_interface name="position"/>
-        <state_interface name="velocity"/>
-        <state_interface name="effort"/>
-      </joint>
+        <command_interface name="effort"/>
+        <state_interface name="position"/>
+        <state_interface name="velocity"/>
+        <state_interface name="effort"/>
+      </joint>
+      <sensor name="${prefix}finger_sensor_4">
+        <state_interface name="Present Pressure 1"/>
+        <state_interface name="Present Pressure 2"/>
+        <state_interface name="Present Pressure 3"/>
+        <state_interface name="Present Pressure 4"/>
+        <state_interface name="Present Pressure 5"/>
+        <state_interface name="Present Pressure 6"/>
+        <state_interface name="Present Pressure 7"/>
+        <state_interface name="Present Pressure 8"/>
+        <state_interface name="Present Pressure 9"/>
+      </sensor>
       <joint name="${prefix}finger_joint_17">
         <command_interface name="position"/>
+        <command_interface name="effort"/>
         <state_interface name="position"/>
         <state_interface name="velocity"/>
@@ -180,4 +241,5 @@
       <joint name="${prefix}finger_joint_18">
         <command_interface name="position"/>
+        <command_interface name="effort"/>
         <state_interface name="position"/>
         <state_interface name="velocity"/>
@@ -186,4 +248,5 @@
       <joint name="${prefix}finger_joint_19">
         <command_interface name="position"/>
+        <command_interface name="effort"/>
         <state_interface name="position"/>
         <state_interface name="velocity"/>
@@ -192,267 +255,539 @@
       <joint name="${prefix}finger_joint_20">
         <command_interface name="position"/>
-        <state_interface name="position"/>
-        <state_interface name="velocity"/>
-        <state_interface name="effort"/>
-      </joint>
+        <command_interface name="effort"/>
+        <state_interface name="position"/>
+        <state_interface name="velocity"/>
+        <state_interface name="effort"/>
+      </joint>
+      <sensor name="${prefix}finger_sensor_5">
+        <state_interface name="Present Pressure 1"/>
+        <state_interface name="Present Pressure 2"/>
+        <state_interface name="Present Pressure 3"/>
+        <state_interface name="Present Pressure 4"/>
+        <state_interface name="Present Pressure 5"/>
+        <state_interface name="Present Pressure 6"/>
+        <state_interface name="Present Pressure 7"/>
+        <state_interface name="Present Pressure 8"/>
+        <state_interface name="Present Pressure 9"/>
+      </sensor>
       <gpio name="dxl1">
         <command_interface name="Goal Position"/>
-        <state_interface name="Present Position"/>
-        <state_interface name="Present Velocity"/>
-        <state_interface name="Present Current"/>
-        <param name="type">dxl</param>
+        <command_interface name="Goal Current"/>
+        <state_interface name="Present Position"/>
+        <state_interface name="Present Velocity"/>
+        <state_interface name="Present Current"/>
+        <param name="type">virtual_dxl</param>
+        <param name="ID">201</param>
+        <param name="comm_id">200</param>
+        <param name="model_num">261</param>
+      </gpio>
+      <gpio name="dxl2">
+        <command_interface name="Goal Position"/>
+        <command_interface name="Goal Current"/>
+        <state_interface name="Present Position"/>
+        <state_interface name="Present Velocity"/>
+        <state_interface name="Present Current"/>
+        <param name="type">virtual_dxl</param>
+        <param name="ID">202</param>
+        <param name="comm_id">200</param>
+        <param name="model_num">262</param>
+      </gpio>
+      <gpio name="dxl3">
+        <command_interface name="Goal Position"/>
+        <command_interface name="Goal Current"/>
+        <state_interface name="Present Position"/>
+        <state_interface name="Present Velocity"/>
+        <state_interface name="Present Current"/>
+        <param name="type">virtual_dxl</param>
+        <param name="ID">203</param>
+        <param name="comm_id">200</param>
+        <param name="model_num">263</param>
+      </gpio>
+      <gpio name="dxl4">
+        <command_interface name="Goal Position"/>
+        <command_interface name="Goal Current"/>
+        <state_interface name="Present Position"/>
+        <state_interface name="Present Velocity"/>
+        <state_interface name="Present Current"/>
+        <param name="type">virtual_dxl</param>
+        <param name="ID">204</param>
+        <param name="comm_id">200</param>
+        <param name="model_num">264</param>
+      </gpio>
+      <gpio name="${prefix}finger_sensor_1">
+        <state_interface name="Present Pressure 1"/>
+        <state_interface name="Present Pressure 2"/>
+        <state_interface name="Present Pressure 3"/>
+        <state_interface name="Present Pressure 4"/>
+        <state_interface name="Present Pressure 5"/>
+        <state_interface name="Present Pressure 6"/>
+        <state_interface name="Present Pressure 7"/>
+        <state_interface name="Present Pressure 8"/>
+        <state_interface name="Present Pressure 9"/>
+        <param name="type">virtual_sensor</param>
+        <param name="ID">205</param>
+        <param name="comm_id">200</param>
+        <param name="model_num">265</param>
+      </gpio>
+      <gpio name="dxl6">
+        <command_interface name="Goal Position"/>
+        <command_interface name="Goal Current"/>
+        <state_interface name="Present Position"/>
+        <state_interface name="Present Velocity"/>
+        <state_interface name="Present Current"/>
+        <param name="type">virtual_dxl</param>
+        <param name="ID">206</param>
+        <param name="comm_id">200</param>
+        <param name="model_num">266</param>
+      </gpio>
+      <gpio name="dxl7">
+        <command_interface name="Goal Position"/>
+        <command_interface name="Goal Current"/>
+        <state_interface name="Present Position"/>
+        <state_interface name="Present Velocity"/>
+        <state_interface name="Present Current"/>
+        <param name="type">virtual_dxl</param>
+        <param name="ID">207</param>
+        <param name="comm_id">200</param>
+        <param name="model_num">267</param>
+      </gpio>
+      <gpio name="dxl8">
+        <command_interface name="Goal Position"/>
+        <command_interface name="Goal Current"/>
+        <state_interface name="Present Position"/>
+        <state_interface name="Present Velocity"/>
+        <state_interface name="Present Current"/>
+        <param name="type">virtual_dxl</param>
+        <param name="ID">208</param>
+        <param name="comm_id">200</param>
+        <param name="model_num">268</param>
+      </gpio>
+      <gpio name="dxl9">
+        <command_interface name="Goal Position"/>
+        <command_interface name="Goal Current"/>
+        <state_interface name="Present Position"/>
+        <state_interface name="Present Velocity"/>
+        <state_interface name="Present Current"/>
+        <param name="type">virtual_dxl</param>
+        <param name="ID">209</param>
+        <param name="comm_id">200</param>
+        <param name="model_num">269</param>
+      </gpio>
+      <gpio name="${prefix}finger_sensor_2">
+        <state_interface name="Present Pressure 1"/>
+        <state_interface name="Present Pressure 2"/>
+        <state_interface name="Present Pressure 3"/>
+        <state_interface name="Present Pressure 4"/>
+        <state_interface name="Present Pressure 5"/>
+        <state_interface name="Present Pressure 6"/>
+        <state_interface name="Present Pressure 7"/>
+        <state_interface name="Present Pressure 8"/>
+        <state_interface name="Present Pressure 9"/>
+        <param name="type">virtual_sensor</param>
+        <param name="ID">210</param>
+        <param name="comm_id">200</param>
+        <param name="model_num">270</param>
+      </gpio>
+      <gpio name="dxl11">
+        <command_interface name="Goal Position"/>
+        <command_interface name="Goal Current"/>
+        <state_interface name="Present Position"/>
+        <state_interface name="Present Velocity"/>
+        <state_interface name="Present Current"/>
+        <param name="type">virtual_dxl</param>
+        <param name="ID">211</param>
+        <param name="comm_id">200</param>
+        <param name="model_num">271</param>
+      </gpio>
+      <gpio name="dxl12">
+        <command_interface name="Goal Position"/>
+        <command_interface name="Goal Current"/>
+        <state_interface name="Present Position"/>
+        <state_interface name="Present Velocity"/>
+        <state_interface name="Present Current"/>
+        <param name="type">virtual_dxl</param>
+        <param name="ID">212</param>
+        <param name="comm_id">200</param>
+        <param name="model_num">272</param>
+      </gpio>
+      <gpio name="dxl13">
+        <command_interface name="Goal Position"/>
+        <command_interface name="Goal Current"/>
+        <state_interface name="Present Position"/>
+        <state_interface name="Present Velocity"/>
+        <state_interface name="Present Current"/>
+        <param name="type">virtual_dxl</param>
+        <param name="ID">213</param>
+        <param name="comm_id">200</param>
+        <param name="model_num">273</param>
+      </gpio>
+      <gpio name="dxl14">
+        <command_interface name="Goal Position"/>
+        <command_interface name="Goal Current"/>
+        <state_interface name="Present Position"/>
+        <state_interface name="Present Velocity"/>
+        <state_interface name="Present Current"/>
+        <param name="type">virtual_dxl</param>
+        <param name="ID">214</param>
+        <param name="comm_id">200</param>
+        <param name="model_num">274</param>
+      </gpio>
+      <gpio name="${prefix}finger_sensor_3">
+        <state_interface name="Present Pressure 1"/>
+        <state_interface name="Present Pressure 2"/>
+        <state_interface name="Present Pressure 3"/>
+        <state_interface name="Present Pressure 4"/>
+        <state_interface name="Present Pressure 5"/>
+        <state_interface name="Present Pressure 6"/>
+        <state_interface name="Present Pressure 7"/>
+        <state_interface name="Present Pressure 8"/>
+        <state_interface name="Present Pressure 9"/>
+        <param name="type">virtual_sensor</param>
+        <param name="ID">215</param>
+        <param name="comm_id">200</param>
+        <param name="model_num">275</param>
+      </gpio>
+      <gpio name="dxl16">
+        <command_interface name="Goal Position"/>
+        <command_interface name="Goal Current"/>
+        <state_interface name="Present Position"/>
+        <state_interface name="Present Velocity"/>
+        <state_interface name="Present Current"/>
+        <param name="type">virtual_dxl</param>
+        <param name="ID">216</param>
+        <param name="comm_id">200</param>
+        <param name="model_num">276</param>
+      </gpio>
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