Commit message: Updated robot naming
Signed-off-by: Hyunwoo Nam <nhw@robotis.com>

File: robotis_hand_description/ros2_control/rh_5_right.ros2_control.xacro (robot description, xacro)
@@ -76,33 +76,33 @@
         </hardware>
       </xacro:unless>
-      <joint name="${prefix}finger_joint_1">
-        <command_interface name="position"/>
-        <command_interface name="effort"/>
-        <state_interface name="position"/>
-        <state_interface name="velocity"/>
-        <state_interface name="effort"/>
-      </joint>
-      <joint name="${prefix}finger_joint_2">
-        <command_interface name="position"/>
-        <command_interface name="effort"/>
-        <state_interface name="position"/>
-        <state_interface name="velocity"/>
-        <state_interface name="effort"/>
-      </joint>
-      <joint name="${prefix}finger_joint_3">
-        <command_interface name="position"/>
-        <command_interface name="effort"/>
-        <state_interface name="position"/>
-        <state_interface name="velocity"/>
-        <state_interface name="effort"/>
-      </joint>
-      <joint name="${prefix}finger_joint_4">
-        <command_interface name="position"/>
-        <command_interface name="effort"/>
-        <state_interface name="position"/>
-        <state_interface name="velocity"/>
-        <state_interface name="effort"/>
-      </joint>
-      <sensor name="${prefix}finger_sensor_1">
+      <joint name="${prefix}finger_r_joint1">
+        <command_interface name="position"/>
+        <command_interface name="effort"/>
+        <state_interface name="position"/>
+        <state_interface name="velocity"/>
+        <state_interface name="effort"/>
+      </joint>
+      <joint name="${prefix}finger_r_joint2">
+        <command_interface name="position"/>
+        <command_interface name="effort"/>
+        <state_interface name="position"/>
+        <state_interface name="velocity"/>
+        <state_interface name="effort"/>
+      </joint>
+      <joint name="${prefix}finger_r_joint3">
+        <command_interface name="position"/>
+        <command_interface name="effort"/>
+        <state_interface name="position"/>
+        <state_interface name="velocity"/>
+        <state_interface name="effort"/>
+      </joint>
+      <joint name="${prefix}finger_r_joint4">
+        <command_interface name="position"/>
+        <command_interface name="effort"/>
+        <state_interface name="position"/>
+        <state_interface name="velocity"/>
+        <state_interface name="effort"/>
+      </joint>
+      <sensor name="${prefix}finger_r_sensor1">
         <state_interface name="Present Pressure 1"/>
         <state_interface name="Present Pressure 2"/>
@@ -115,33 +115,33 @@
         <state_interface name="Present Pressure 9"/>
       </sensor>
-      <joint name="${prefix}finger_joint_5">
-        <command_interface name="position"/>
-        <command_interface name="effort"/>
-        <state_interface name="position"/>
-        <state_interface name="velocity"/>
-        <state_interface name="effort"/>
-      </joint>
-      <joint name="${prefix}finger_joint_6">
-        <command_interface name="position"/>
-        <command_interface name="effort"/>
-        <state_interface name="position"/>
-        <state_interface name="velocity"/>
-        <state_interface name="effort"/>
-      </joint>
-      <joint name="${prefix}finger_joint_7">
-        <command_interface name="position"/>
-        <command_interface name="effort"/>
-        <state_interface name="position"/>
-        <state_interface name="velocity"/>
-        <state_interface name="effort"/>
-      </joint>
-      <joint name="${prefix}finger_joint_8">
-        <command_interface name="position"/>
-        <command_interface name="effort"/>
-        <state_interface name="position"/>
-        <state_interface name="velocity"/>
-        <state_interface name="effort"/>
-      </joint>
-      <sensor name="${prefix}finger_sensor_2">
+      <joint name="${prefix}finger_r_joint5">
+        <command_interface name="position"/>
+        <command_interface name="effort"/>
+        <state_interface name="position"/>
+        <state_interface name="velocity"/>
+        <state_interface name="effort"/>
+      </joint>
+      <joint name="${prefix}finger_r_joint6">
+        <command_interface name="position"/>
+        <command_interface name="effort"/>
+        <state_interface name="position"/>
+        <state_interface name="velocity"/>
+        <state_interface name="effort"/>
+      </joint>
+      <joint name="${prefix}finger_r_joint7">
+        <command_interface name="position"/>
+        <command_interface name="effort"/>
+        <state_interface name="position"/>
+        <state_interface name="velocity"/>
+        <state_interface name="effort"/>
+      </joint>
+      <joint name="${prefix}finger_r_joint8">
+        <command_interface name="position"/>
+        <command_interface name="effort"/>
+        <state_interface name="position"/>
+        <state_interface name="velocity"/>
+        <state_interface name="effort"/>
+      </joint>
+      <sensor name="${prefix}finger_r_sensor2">
         <state_interface name="Present Pressure 1"/>
         <state_interface name="Present Pressure 2"/>
@@ -154,33 +154,33 @@
         <state_interface name="Present Pressure 9"/>
       </sensor>
-      <joint name="${prefix}finger_joint_9">
-        <command_interface name="position"/>
-        <command_interface name="effort"/>
-        <state_interface name="position"/>
-        <state_interface name="velocity"/>
-        <state_interface name="effort"/>
-      </joint>
-      <joint name="${prefix}finger_joint_10">
-        <command_interface name="position"/>
-        <command_interface name="effort"/>
-        <state_interface name="position"/>
-        <state_interface name="velocity"/>
-        <state_interface name="effort"/>
-      </joint>
-      <joint name="${prefix}finger_joint_11">
-        <command_interface name="position"/>
-        <command_interface name="effort"/>
-        <state_interface name="position"/>
-        <state_interface name="velocity"/>
-        <state_interface name="effort"/>
-      </joint>
-      <joint name="${prefix}finger_joint_12">
-        <command_interface name="position"/>
-        <command_interface name="effort"/>
-        <state_interface name="position"/>
-        <state_interface name="velocity"/>
-        <state_interface name="effort"/>
-      </joint>
-      <sensor name="${prefix}finger_sensor_3">
+      <joint name="${prefix}finger_r_joint9">
+        <command_interface name="position"/>
+        <command_interface name="effort"/>
+        <state_interface name="position"/>
+        <state_interface name="velocity"/>
+        <state_interface name="effort"/>
+      </joint>
+      <joint name="${prefix}finger_r_joint10">
+        <command_interface name="position"/>
+        <command_interface name="effort"/>
+        <state_interface name="position"/>
+        <state_interface name="velocity"/>
+        <state_interface name="effort"/>
+      </joint>
+      <joint name="${prefix}finger_r_joint11">
+        <command_interface name="position"/>
+        <command_interface name="effort"/>
+        <state_interface name="position"/>
+        <state_interface name="velocity"/>
+        <state_interface name="effort"/>
+      </joint>
+      <joint name="${prefix}finger_r_joint12">
+        <command_interface name="position"/>
+        <command_interface name="effort"/>
+        <state_interface name="position"/>
+        <state_interface name="velocity"/>
+        <state_interface name="effort"/>
+      </joint>
+      <sensor name="${prefix}finger_r_sensor3">
         <state_interface name="Present Pressure 1"/>
         <state_interface name="Present Pressure 2"/>
@@ -193,33 +193,33 @@
         <state_interface name="Present Pressure 9"/>
       </sensor>
-      <joint name="${prefix}finger_joint_13">
-        <command_interface name="position"/>
-        <command_interface name="effort"/>
-        <state_interface name="position"/>
-        <state_interface name="velocity"/>
-        <state_interface name="effort"/>
-      </joint>
-      <joint name="${prefix}finger_joint_14">
-        <command_interface name="position"/>
-        <command_interface name="effort"/>
-        <state_interface name="position"/>
-        <state_interface name="velocity"/>
-        <state_interface name="effort"/>
-      </joint>
-      <joint name="${prefix}finger_joint_15">
-        <command_interface name="position"/>
-        <command_interface name="effort"/>
-        <state_interface name="position"/>
-        <state_interface name="velocity"/>
-        <state_interface name="effort"/>
-      </joint>
-      <joint name="${prefix}finger_joint_16">
-        <command_interface name="position"/>
-        <command_interface name="effort"/>
-        <state_interface name="position"/>
-        <state_interface name="velocity"/>
-        <state_interface name="effort"/>
-      </joint>
-      <sensor name="${prefix}finger_sensor_4">
+      <joint name="${prefix}finger_r_joint13">
+        <command_interface name="position"/>
+        <command_interface name="effort"/>
+        <state_interface name="position"/>
+        <state_interface name="velocity"/>
+        <state_interface name="effort"/>
+      </joint>
+      <joint name="${prefix}finger_r_joint14">
+        <command_interface name="position"/>
+        <command_interface name="effort"/>
+        <state_interface name="position"/>
+        <state_interface name="velocity"/>
+        <state_interface name="effort"/>
+      </joint>
+      <joint name="${prefix}finger_r_joint15">
+        <command_interface name="position"/>
+        <command_interface name="effort"/>
+        <state_interface name="position"/>
+        <state_interface name="velocity"/>
+        <state_interface name="effort"/>
+      </joint>
+      <joint name="${prefix}finger_r_joint16">
+        <command_interface name="position"/>
+        <command_interface name="effort"/>
+        <state_interface name="position"/>
+        <state_interface name="velocity"/>
+        <state_interface name="effort"/>
+      </joint>
+      <sensor name="${prefix}finger_r_sensor4">
         <state_interface name="Present Pressure 1"/>
         <state_interface name="Present Pressure 2"/>
@@ -232,33 +232,33 @@
         <state_interface name="Present Pressure 9"/>
       </sensor>
-      <joint name="${prefix}finger_joint_17">
-        <command_interface name="position"/>
-        <command_interface name="effort"/>
-        <state_interface name="position"/>
-        <state_interface name="velocity"/>
-        <state_interface name="effort"/>
-      </joint>
-      <joint name="${prefix}finger_joint_18">
-        <command_interface name="position"/>
-        <command_interface name="effort"/>
-        <state_interface name="position"/>
-        <state_interface name="velocity"/>
-        <state_interface name="effort"/>
-      </joint>
-      <joint name="${prefix}finger_joint_19">
-        <command_interface name="position"/>
-        <command_interface name="effort"/>
-        <state_interface name="position"/>
-        <state_interface name="velocity"/>
-        <state_interface name="effort"/>
-      </joint>
-      <joint name="${prefix}finger_joint_20">
-        <command_interface name="position"/>
-        <command_interface name="effort"/>
-        <state_interface name="position"/>
-        <state_interface name="velocity"/>
-        <state_interface name="effort"/>
-      </joint>
-      <sensor name="${prefix}finger_sensor_5">
+      <joint name="${prefix}finger_r_joint17">
+        <command_interface name="position"/>
+        <command_interface name="effort"/>
+        <state_interface name="position"/>
+        <state_interface name="velocity"/>
+        <state_interface name="effort"/>
+      </joint>
+      <joint name="${prefix}finger_r_joint18">
+        <command_interface name="position"/>
+        <command_interface name="effort"/>
+        <state_interface name="position"/>
+        <state_interface name="velocity"/>
+        <state_interface name="effort"/>
+      </joint>
+      <joint name="${prefix}finger_r_joint19">
+        <command_interface name="position"/>
+        <command_interface name="effort"/>
+        <state_interface name="position"/>
+        <state_interface name="velocity"/>
+        <state_interface name="effort"/>
+      </joint>
+      <joint name="${prefix}finger_r_joint20">
+        <command_interface name="position"/>
+        <command_interface name="effort"/>
+        <state_interface name="position"/>
+        <state_interface name="velocity"/>
+        <state_interface name="effort"/>
+      </joint>
+      <sensor name="${prefix}finger_r_sensor5">
         <state_interface name="Present Pressure 1"/>
         <state_interface name="Present Pressure 2"/>
@@ -271,5 +271,5 @@
         <state_interface name="Present Pressure 9"/>
       </sensor>
-      <!-- <gpio name="dxl1">
+      <gpio name="dxl1">
         <command_interface name="Goal Position"/>
         <command_interface name="Goal Current"/>
@@ -315,5 +315,5 @@
         <param name="model_num">264</param>
       </gpio>
-      <gpio name="${prefix}finger_sensor_1">
+      <gpio name="${prefix}finger_r_sensor1">
         <state_interface name="Present Pressure 1"/>
         <state_interface name="Present Pressure 2"/>
@@ -374,5 +374,5 @@
         <param name="model_num">269</param>
       </gpio>
-      <gpio name="${prefix}finger_sensor_2">
+      <gpio name="${prefix}finger_r_sensor2">
         <state_interface name="Present Pressure 1"/>
         <state_interface name="Present Pressure 2"/>
@@ -433,5 +433,5 @@
         <param name="model_num">274</param>
       </gpio>
-      <gpio name="${prefix}finger_sensor_3">
+      <gpio name="${prefix}finger_r_sensor3">
         <state_interface name="Present Pressure 1"/>
         <state_interface name="Present Pressure 2"/>
@@ -492,5 +492,5 @@
         <param name="model_num">279</param>
       </gpio>
-      <gpio name="${prefix}finger_sensor_4">
+      <gpio name="${prefix}finger_r_sensor4">
         <state_interface name="Present Pressure 1"/>
         <state_interface name="Present Pressure 2"/>
@@ -551,5 +551,5 @@
         <param name="model_num">284</param>
       </gpio>
-      <gpio name="${prefix}finger_sensor_5">
+      <gpio name="${prefix}finger_r_sensor5">
         <state_interface name="Present Pressure 1"/>
         <state_interface name="Present Pressure 2"/>
@@ -776,519 +776,4 @@
       </gpio>
       <gpio name="dxl24_init">
-        <param name="type">controller</param>
-        <param name="ID">24</param>
-        <param name="Position P Gain">1600</param>
-        <param name="Position D Gain">5000</param>
-        <param name="Startup Configuration">2</param>
-        <param name="Drive Mode">12</param>
-        <param name="Bus Watchdog">0</param>
-        <param name="Profile Velocity">20</param>
-        <param name="Profile Acceleration">10</param>
-      </gpio> -->
-      <gpio name="dxl226">
-        <command_interface name="Goal Position"/>
-        <command_interface name="Goal Current"/>
-        <state_interface name="Present Position"/>
-        <state_interface name="Present Velocity"/>
-        <state_interface name="Present Current"/>
-        <param name="type">virtual_dxl</param>
-        <param name="ID">201</param>
-        <param name="comm_id">200</param>
-        <param name="model_num">261</param>
-      </gpio>
-      <gpio name="dxl227">
-        <command_interface name="Goal Position"/>
-        <command_interface name="Goal Current"/>
-        <state_interface name="Present Position"/>
-        <state_interface name="Present Velocity"/>
-        <state_interface name="Present Current"/>
-        <param name="type">virtual_dxl</param>
-        <param name="ID">202</param>
-        <param name="comm_id">200</param>
-        <param name="model_num">262</param>
-      </gpio>
-      <gpio name="dxl228">
-        <command_interface name="Goal Position"/>
-        <command_interface name="Goal Current"/>
-        <state_interface name="Present Position"/>
-        <state_interface name="Present Velocity"/>
-        <state_interface name="Present Current"/>
-        <param name="type">virtual_dxl</param>
-        <param name="ID">203</param>
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
File: robotis_hand_description/urdf/rh_5_left.xacro (robot description, xacro)
@@ -7,5 +7,5 @@
   <xacro:include filename="$(find robotis_hand_description)/urdf/rh_5_left.urdf.xacro" />
   <xacro:include filename="$(find robotis_hand_description)/gazebo/robotis_hand.gazebo.xacro" />
-  <xacro:include filename="$(find robotis_hand_description)/ros2_control/robotis_hand.ros2_control.xacro" />
+  <xacro:include filename="$(find robotis_hand_description)/ros2_control/rh_5_left.ros2_control.xacro" />
   <link name="world"/>
   <joint name="$(arg prefix)world_fixed" type="fixed">

File: robotis_hand_description/urdf/rh_5_right.xacro (robot description, xacro)
@@ -7,5 +7,5 @@
   <xacro:include filename="$(find robotis_hand_description)/urdf/rh_5_right.urdf.xacro" />
   <xacro:include filename="$(find robotis_hand_description)/gazebo/robotis_hand.gazebo.xacro" />
-  <xacro:include filename="$(find robotis_hand_description)/ros2_control/robotis_hand.ros2_control.xacro" />
+  <xacro:include filename="$(find robotis_hand_description)/ros2_control/rh_5_right.ros2_control.xacro" />
   <link name="world"/>
   <joint name="$(arg prefix)world_fixed" type="fixed">
