Commit message: Add tactile model configuration and pressure sensor updates
- Added new YAML configuration files for pressure sensors (pressure_9.yaml and pressure_10.yaml) to support different channel counts.
- Updated the hx5_d20_hardware_controller_manager.yaml to remove references to the now obsolete Present Pressure 10.
- Enhanced launch files (hx5_d20_left.launch.py and hx5_d20_right.launch.py) to include new launch arguments for tactile model profiles and number of taxels.
- Introduced tactile_model.py for managing tactile layouts and resolving sensor configurations.
- Added tests for tactile configuration and model validation to ensure compatibility with hardware setups.

File: robotis_hand_description/ros2_control/hx5_d20_rev1/hx5_d20_left.ros2_control.xacro (robot description, xacro)
@@ -1,5 +1,5 @@
 <?xml version="1.0"?>
 <robot xmlns:xacro="http://www.ros.org/wiki/xacro">
-  <xacro:macro name="hx5_left_system" params="name prefix port_name:=^|/dev/ttyUSB0 use_sim:=^|false use_mock_hardware:=^|false mock_sensor_commands:=^|false">
+  <xacro:macro name="hx5_left_system" params="name prefix port_name:=^|/dev/ttyUSB0 use_sim:=^|false use_mock_hardware:=^|false mock_sensor_commands:=^|false num_taxels:=9">
     <ros2_control name="${name}" type="system" is_async="true">
       <xacro:if value="$(arg use_sim)">
@@ -70,4 +70,7 @@
         <state_interface name="Present Pressure 8"/>
         <state_interface name="Present Pressure 9"/>
+        <xacro:if value="${int(num_taxels) == 10}">
+          <state_interface name="Present Pressure 10"/>
+        </xacro:if>
       </sensor>
       <joint name="${prefix}finger_l_joint5">
@@ -109,4 +112,7 @@
         <state_interface name="Present Pressure 8"/>
         <state_interface name="Present Pressure 9"/>
+        <xacro:if value="${int(num_taxels) == 10}">
+          <state_interface name="Present Pressure 10"/>
+        </xacro:if>
       </sensor>
       <joint name="${prefix}finger_l_joint9">
@@ -148,4 +154,7 @@
         <state_interface name="Present Pressure 8"/>
         <state_interface name="Present Pressure 9"/>
+        <xacro:if value="${int(num_taxels) == 10}">
+          <state_interface name="Present Pressure 10"/>
+        </xacro:if>
       </sensor>
       <joint name="${prefix}finger_l_joint13">
@@ -187,4 +196,7 @@
         <state_interface name="Present Pressure 8"/>
         <state_interface name="Present Pressure 9"/>
+        <xacro:if value="${int(num_taxels) == 10}">
+          <state_interface name="Present Pressure 10"/>
+        </xacro:if>
       </sensor>
       <joint name="${prefix}finger_l_joint17">
@@ -226,4 +238,7 @@
         <state_interface name="Present Pressure 8"/>
         <state_interface name="Present Pressure 9"/>
+        <xacro:if value="${int(num_taxels) == 10}">
+          <state_interface name="Present Pressure 10"/>
+        </xacro:if>
       </sensor>
       <gpio name="hand_l_controller">
@@ -267,5 +282,5 @@
         <param name="SyncTable 1 Read Size 3">6</param>
         <param name="SyncTable 1 Read Size 4">6</param>
-        <param name="SyncTable 1 Read Size 5">9</param>
+        <param name="SyncTable 1 Read Size 5">${num_taxels}</param>
         <param name="SyncTable 1 Write Address 1">230</param>
         <param name="SyncTable 1 Write Address 2">230</param>
@@ -287,5 +302,5 @@
         <param name="SyncTable 2 Read Size 3">6</param>
         <param name="SyncTable 2 Read Size 4">6</param>
-        <param name="SyncTable 2 Read Size 5">9</param>
+        <param name="SyncTable 2 Read Size 5">${num_taxels}</param>
         <param name="SyncTable 2 Write Address 1">230</param>
         <param name="SyncTable 2 Write Address 2">230</param>
@@ -307,5 +322,5 @@
         <param name="SyncTable 3 Read Size 3">6</param>
         <param name="SyncTable 3 Read Size 4">6</param>
-        <param name="SyncTable 3 Read Size 5">9</param>
+        <param name="SyncTable 3 Read Size 5">${num_taxels}</param>
         <param name="SyncTable 3 Write Address 1">230</param>
         <param name="SyncTable 3 Write Address 2">230</param>
@@ -327,5 +342,5 @@
         <param name="SyncTable 4 Read Size 3">6</param>
         <param name="SyncTable 4 Read Size 4">6</param>
-        <param name="SyncTable 4 Read Size 5">9</param>
+        <param name="SyncTable 4 Read Size 5">${num_taxels}</param>
         <param name="SyncTable 4 Write Address 1">230</param>
         <param name="SyncTable 4 Write Address 2">230</param>
@@ -347,5 +362,5 @@
         <param name="SyncTable 5 Read Size 3">6</param>
         <param name="SyncTable 5 Read Size 4">6</param>
-        <param name="SyncTable 5 Read Size 5">9</param>
+        <param name="SyncTable 5 Read Size 5">${num_taxels}</param>
         <param name="SyncTable 5 Write Address 1">230</param>
         <param name="SyncTable 5 Write Address 2">230</param>
@@ -887,4 +902,7 @@
         <state_interface name="Present Pressure 8"/>
         <state_interface name="Present Pressure 9"/>
+        <xacro:if value="${int(num_taxels) == 10}">
+          <state_interface name="Present Pressure 10"/>
+        </xacro:if>
         <param name="type">virtual_sensor</param>
         <param name="ID">145</param>
@@ -946,4 +964,7 @@
         <state_interface name="Present Pressure 8"/>
         <state_interface name="Present Pressure 9"/>
+        <xacro:if value="${int(num_taxels) == 10}">
+          <state_interface name="Present Pressure 10"/>
+        </xacro:if>
         <param name="type">virtual_sensor</param>
         <param name="ID">150</param>
@@ -1005,4 +1026,7 @@
         <state_interface name="Present Pressure 8"/>
         <state_interface name="Present Pressure 9"/>
+        <xacro:if value="${int(num_taxels) == 10}">
+          <state_interface name="Present Pressure 10"/>
+        </xacro:if>
         <param name="type">virtual_sensor</param>
         <param name="ID">155</param>
@@ -1064,4 +1088,7 @@
         <state_interface name="Present Pressure 8"/>
         <state_interface name="Present Pressure 9"/>
+        <xacro:if value="${int(num_taxels) == 10}">
+          <state_interface name="Present Pressure 10"/>
+        </xacro:if>
         <param name="type">virtual_sensor</param>
         <param name="ID">160</param>
@@ -1123,4 +1150,7 @@
         <state_interface name="Present Pressure 8"/>
         <state_interface name="Present Pressure 9"/>
+        <xacro:if value="${int(num_taxels) == 10}">
+          <state_interface name="Present Pressure 10"/>
+        </xacro:if>
         <param name="type">virtual_sensor</param>
         <param name="ID">165</param>

File: robotis_hand_description/ros2_control/hx5_d20_rev1/hx5_d20_right.ros2_control.xacro (robot description, xacro)
@@ -1,5 +1,5 @@
 <?xml version="1.0"?>
 <robot xmlns:xacro="http://www.ros.org/wiki/xacro">
-  <xacro:macro name="hx5_right_system" params="name prefix port_name:=^|/dev/ttyUSB0 use_sim:=^|false use_mock_hardware:=^|false mock_sensor_commands:=^|false">
+  <xacro:macro name="hx5_right_system" params="name prefix port_name:=^|/dev/ttyUSB0 use_sim:=^|false use_mock_hardware:=^|false mock_sensor_commands:=^|false num_taxels:=9">
     <ros2_control name="${name}" type="system" is_async="true">
       <xacro:if value="$(arg use_sim)">
@@ -70,4 +70,7 @@
         <state_interface name="Present Pressure 8"/>
         <state_interface name="Present Pressure 9"/>
+        <xacro:if value="${int(num_taxels) == 10}">
+          <state_interface name="Present Pressure 10"/>
+        </xacro:if>
       </sensor>
       <joint name="${prefix}finger_r_joint5">
@@ -109,4 +112,7 @@
         <state_interface name="Present Pressure 8"/>
         <state_interface name="Present Pressure 9"/>
+        <xacro:if value="${int(num_taxels) == 10}">
+          <state_interface name="Present Pressure 10"/>
+        </xacro:if>
       </sensor>
       <joint name="${prefix}finger_r_joint9">
@@ -148,4 +154,7 @@
         <state_interface name="Present Pressure 8"/>
         <state_interface name="Present Pressure 9"/>
+        <xacro:if value="${int(num_taxels) == 10}">
+          <state_interface name="Present Pressure 10"/>
+        </xacro:if>
       </sensor>
       <joint name="${prefix}finger_r_joint13">
@@ -187,4 +196,7 @@
         <state_interface name="Present Pressure 8"/>
         <state_interface name="Present Pressure 9"/>
+        <xacro:if value="${int(num_taxels) == 10}">
+          <state_interface name="Present Pressure 10"/>
+        </xacro:if>
       </sensor>
       <joint name="${prefix}finger_r_joint17">
@@ -226,4 +238,7 @@
         <state_interface name="Present Pressure 8"/>
         <state_interface name="Present Pressure 9"/>
+        <xacro:if value="${int(num_taxels) == 10}">
+          <state_interface name="Present Pressure 10"/>
+        </xacro:if>
       </sensor>
       <gpio name="hand_r_controller">
@@ -267,5 +282,5 @@
         <param name="SyncTable 1 Read Size 3">6</param>
         <param name="SyncTable 1 Read Size 4">6</param>
-        <param name="SyncTable 1 Read Size 5">9</param>
+        <param name="SyncTable 1 Read Size 5">${num_taxels}</param>
         <param name="SyncTable 1 Write Address 1">230</param>
         <param name="SyncTable 1 Write Address 2">230</param>
@@ -287,5 +302,5 @@
         <param name="SyncTable 2 Read Size 3">6</param>
         <param name="SyncTable 2 Read Size 4">6</param>
-        <param name="SyncTable 2 Read Size 5">9</param>
+        <param name="SyncTable 2 Read Size 5">${num_taxels}</param>
         <param name="SyncTable 2 Write Address 1">230</param>
         <param name="SyncTable 2 Write Address 2">230</param>
@@ -307,5 +322,5 @@
         <param name="SyncTable 3 Read Size 3">6</param>
         <param name="SyncTable 3 Read Size 4">6</param>
-        <param name="SyncTable 3 Read Size 5">9</param>
+        <param name="SyncTable 3 Read Size 5">${num_taxels}</param>
         <param name="SyncTable 3 Write Address 1">230</param>
         <param name="SyncTable 3 Write Address 2">230</param>
@@ -327,5 +342,5 @@
         <param name="SyncTable 4 Read Size 3">6</param>
         <param name="SyncTable 4 Read Size 4">6</param>
-        <param name="SyncTable 4 Read Size 5">9</param>
+        <param name="SyncTable 4 Read Size 5">${num_taxels}</param>
         <param name="SyncTable 4 Write Address 1">230</param>
         <param name="SyncTable 4 Write Address 2">230</param>
@@ -347,5 +362,5 @@
         <param name="SyncTable 5 Read Size 3">6</param>
         <param name="SyncTable 5 Read Size 4">6</param>
-        <param name="SyncTable 5 Read Size 5">9</param>
+        <param name="SyncTable 5 Read Size 5">${num_taxels}</param>
         <param name="SyncTable 5 Write Address 1">230</param>
         <param name="SyncTable 5 Write Address 2">230</param>
@@ -887,4 +902,7 @@
         <state_interface name="Present Pressure 8"/>
         <state_interface name="Present Pressure 9"/>
+        <xacro:if value="${int(num_taxels) == 10}">
+          <state_interface name="Present Pressure 10"/>
+        </xacro:if>
         <param name="type">virtual_sensor</param>
         <param name="ID">115</param>
@@ -946,4 +964,7 @@
         <state_interface name="Present Pressure 8"/>
         <state_interface name="Present Pressure 9"/>
+        <xacro:if value="${int(num_taxels) == 10}">
+          <state_interface name="Present Pressure 10"/>
+        </xacro:if>
         <param name="type">virtual_sensor</param>
         <param name="ID">120</param>
@@ -1005,4 +1026,7 @@
         <state_interface name="Present Pressure 8"/>
         <state_interface name="Present Pressure 9"/>
+        <xacro:if value="${int(num_taxels) == 10}">
+          <state_interface name="Present Pressure 10"/>
+        </xacro:if>
         <param name="type">virtual_sensor</param>
         <param name="ID">125</param>
@@ -1064,4 +1088,7 @@
         <state_interface name="Present Pressure 8"/>
         <state_interface name="Present Pressure 9"/>
+        <xacro:if value="${int(num_taxels) == 10}">
+          <state_interface name="Present Pressure 10"/>
+        </xacro:if>
         <param name="type">virtual_sensor</param>
         <param name="ID">130</param>
@@ -1123,4 +1150,7 @@
         <state_interface name="Present Pressure 8"/>
         <state_interface name="Present Pressure 9"/>
+        <xacro:if value="${int(num_taxels) == 10}">
+          <state_interface name="Present Pressure 10"/>
+        </xacro:if>
         <param name="type">virtual_sensor</param>
         <param name="ID">135</param>

File: robotis_hand_description/ros2_control/hx5_d20_rev2/hx5_d20_left.ros2_control.xacro (robot description, xacro)
@@ -1,5 +1,5 @@
 <?xml version="1.0"?>
 <robot xmlns:xacro="http://www.ros.org/wiki/xacro">
-  <xacro:macro name="hx5_left_system" params="name prefix port_name:=^|/dev/ttyUSB0 use_sim:=^|false use_mock_hardware:=^|false mock_sensor_commands:=^|false">
+  <xacro:macro name="hx5_left_system" params="name prefix port_name:=^|/dev/ttyUSB0 use_sim:=^|false use_mock_hardware:=^|false mock_sensor_commands:=^|false num_taxels:=9">
     <ros2_control name="${name}" type="system" is_async="true">
       <xacro:if value="$(arg use_sim)">
@@ -70,4 +70,7 @@
         <state_interface name="Present Pressure 8"/>
         <state_interface name="Present Pressure 9"/>
+        <xacro:if value="${int(num_taxels) == 10}">
+          <state_interface name="Present Pressure 10"/>
+        </xacro:if>
       </sensor>
       <joint name="${prefix}finger_l_joint5">
@@ -109,4 +112,7 @@
         <state_interface name="Present Pressure 8"/>
         <state_interface name="Present Pressure 9"/>
+        <xacro:if value="${int(num_taxels) == 10}">
+          <state_interface name="Present Pressure 10"/>
+        </xacro:if>
       </sensor>
       <joint name="${prefix}finger_l_joint9">
@@ -148,4 +154,7 @@
         <state_interface name="Present Pressure 8"/>
         <state_interface name="Present Pressure 9"/>
+        <xacro:if value="${int(num_taxels) == 10}">
+          <state_interface name="Present Pressure 10"/>
+        </xacro:if>
       </sensor>
       <joint name="${prefix}finger_l_joint13">
@@ -187,4 +196,7 @@
         <state_interface name="Present Pressure 8"/>
         <state_interface name="Present Pressure 9"/>
+        <xacro:if value="${int(num_taxels) == 10}">
+          <state_interface name="Present Pressure 10"/>
+        </xacro:if>
       </sensor>
       <joint name="${prefix}finger_l_joint17">
@@ -226,4 +238,7 @@
         <state_interface name="Present Pressure 8"/>
         <state_interface name="Present Pressure 9"/>
+        <xacro:if value="${int(num_taxels) == 10}">
+          <state_interface name="Present Pressure 10"/>
+        </xacro:if>
       </sensor>
       <gpio name="hand_l_controller">
@@ -267,5 +282,5 @@
         <param name="SyncTable 1 Read Size 3">6</param>
         <param name="SyncTable 1 Read Size 4">6</param>
-        <param name="SyncTable 1 Read Size 5">9</param>
+        <param name="SyncTable 1 Read Size 5">${num_taxels}</param>
         <param name="SyncTable 1 Write Address 1">230</param>
         <param name="SyncTable 1 Write Address 2">230</param>
@@ -287,5 +302,5 @@
         <param name="SyncTable 2 Read Size 3">6</param>
         <param name="SyncTable 2 Read Size 4">6</param>
-        <param name="SyncTable 2 Read Size 5">9</param>
+        <param name="SyncTable 2 Read Size 5">${num_taxels}</param>
         <param name="SyncTable 2 Write Address 1">230</param>
         <param name="SyncTable 2 Write Address 2">230</param>
@@ -307,5 +322,5 @@
         <param name="SyncTable 3 Read Size 3">6</param>
         <param name="SyncTable 3 Read Size 4">6</param>
-        <param name="SyncTable 3 Read Size 5">9</param>
+        <param name="SyncTable 3 Read Size 5">${num_taxels}</param>
         <param name="SyncTable 3 Write Address 1">230</param>
         <param name="SyncTable 3 Write Address 2">230</param>
@@ -327,5 +342,5 @@
         <param name="SyncTable 4 Read Size 3">6</param>
         <param name="SyncTable 4 Read Size 4">6</param>
-        <param name="SyncTable 4 Read Size 5">9</param>
+        <param name="SyncTable 4 Read Size 5">${num_taxels}</param>
         <param name="SyncTable 4 Write Address 1">230</param>
         <param name="SyncTable 4 Write Address 2">230</param>
@@ -347,5 +362,5 @@
         <param name="SyncTable 5 Read Size 3">6</param>
         <param name="SyncTable 5 Read Size 4">6</param>
-        <param name="SyncTable 5 Read Size 5">9</param>
+        <param name="SyncTable 5 Read Size 5">${num_taxels}</param>
         <param name="SyncTable 5 Write Address 1">230</param>
         <param name="SyncTable 5 Write Address 2">230</param>
@@ -887,4 +902,7 @@
         <state_interface name="Present Pressure 8"/>
         <state_interface name="Present Pressure 9"/>
+        <xacro:if value="${int(num_taxels) == 10}">
+          <state_interface name="Present Pressure 10"/>
+        </xacro:if>
         <param name="type">virtual_sensor</param>
         <param name="ID">145</param>
@@ -946,4 +964,7 @@
         <state_interface name="Present Pressure 8"/>
         <state_interface name="Present Pressure 9"/>
+        <xacro:if value="${int(num_taxels) == 10}">
+          <state_interface name="Present Pressure 10"/>
+        </xacro:if>
         <param name="type">virtual_sensor</param>
         <param name="ID">150</param>
@@ -1005,4 +1026,7 @@
         <state_interface name="Present Pressure 8"/>
         <state_interface name="Present Pressure 9"/>
+        <xacro:if value="${int(num_taxels) == 10}">
+          <state_interface name="Present Pressure 10"/>
+        </xacro:if>
         <param name="type">virtual_sensor</param>
         <param name="ID">155</param>
@@ -1064,4 +1088,7 @@
         <state_interface name="Present Pressure 8"/>
         <state_interface name="Present Pressure 9"/>
+        <xacro:if value="${int(num_taxels) == 10}">
+          <state_interface name="Present Pressure 10"/>
+        </xacro:if>
         <param name="type">virtual_sensor</param>
         <param name="ID">160</param>
@@ -1123,4 +1150,7 @@
         <state_interface name="Present Pressure 8"/>
         <state_interface name="Present Pressure 9"/>
+        <xacro:if value="${int(num_taxels) == 10}">
+          <state_interface name="Present Pressure 10"/>
+        </xacro:if>
         <param name="type">virtual_sensor</param>
         <param name="ID">165</param>
