Commit message: Add tactile model configuration and pressure sensor updates
- Added new YAML configuration files for pressure sensors (pressure_9.yaml and pressure_10.yaml) to support different channel counts.
- Updated the hx5_d20_hardware_controller_manager.yaml to remove references to the now obsolete Present Pressure 10.
- Enhanced launch files (hx5_d20_left.launch.py and hx5_d20_right.launch.py) to include new launch arguments for tactile model profiles and number of taxels.
- Introduced tactile_model.py for managing tactile layouts and resolving sensor configurations.
- Added tests for tactile configuration and model validation to ensure compatibility with hardware setups.

File: robotis_hand_description/ros2_control/hx5_d20_rev2/hx5_d20_right.ros2_control.xacro (robot description, xacro)
@@ -1,5 +1,5 @@
 <?xml version="1.0"?>
 <robot xmlns:xacro="http://www.ros.org/wiki/xacro">
-  <xacro:macro name="hx5_right_system" params="name prefix port_name:=^|/dev/ttyUSB0 use_sim:=^|false use_mock_hardware:=^|false mock_sensor_commands:=^|false">
+  <xacro:macro name="hx5_right_system" params="name prefix port_name:=^|/dev/ttyUSB0 use_sim:=^|false use_mock_hardware:=^|false mock_sensor_commands:=^|false num_taxels:=9">
     <ros2_control name="${name}" type="system" is_async="true">
       <xacro:if value="$(arg use_sim)">
@@ -70,5 +70,7 @@
         <state_interface name="Present Pressure 8"/>
         <state_interface name="Present Pressure 9"/>
-        <state_interface name="Present Pressure 10"/>
+        <xacro:if value="${int(num_taxels) == 10}">
+          <state_interface name="Present Pressure 10"/>
+        </xacro:if>
       </sensor>
       <joint name="${prefix}finger_r_joint5">
@@ -110,5 +112,7 @@
         <state_interface name="Present Pressure 8"/>
         <state_interface name="Present Pressure 9"/>
-        <state_interface name="Present Pressure 10"/>
+        <xacro:if value="${int(num_taxels) == 10}">
+          <state_interface name="Present Pressure 10"/>
+        </xacro:if>
       </sensor>
       <joint name="${prefix}finger_r_joint9">
@@ -150,5 +154,7 @@
         <state_interface name="Present Pressure 8"/>
         <state_interface name="Present Pressure 9"/>
-        <state_interface name="Present Pressure 10"/>
+        <xacro:if value="${int(num_taxels) == 10}">
+          <state_interface name="Present Pressure 10"/>
+        </xacro:if>
       </sensor>
       <joint name="${prefix}finger_r_joint13">
@@ -190,5 +196,7 @@
         <state_interface name="Present Pressure 8"/>
         <state_interface name="Present Pressure 9"/>
-        <state_interface name="Present Pressure 10"/>
+        <xacro:if value="${int(num_taxels) == 10}">
+          <state_interface name="Present Pressure 10"/>
+        </xacro:if>
       </sensor>
       <joint name="${prefix}finger_r_joint17">
@@ -230,5 +238,7 @@
         <state_interface name="Present Pressure 8"/>
         <state_interface name="Present Pressure 9"/>
-        <state_interface name="Present Pressure 10"/>
+        <xacro:if value="${int(num_taxels) == 10}">
+          <state_interface name="Present Pressure 10"/>
+        </xacro:if>
       </sensor>
       <gpio name="hand_r_controller">
@@ -272,5 +282,5 @@
         <param name="SyncTable 1 Read Size 3">6</param>
         <param name="SyncTable 1 Read Size 4">6</param>
-        <param name="SyncTable 1 Read Size 5">10</param>
+        <param name="SyncTable 1 Read Size 5">${num_taxels}</param>
         <param name="SyncTable 1 Write Address 1">230</param>
         <param name="SyncTable 1 Write Address 2">230</param>
@@ -292,5 +302,5 @@
         <param name="SyncTable 2 Read Size 3">6</param>
         <param name="SyncTable 2 Read Size 4">6</param>
-        <param name="SyncTable 2 Read Size 5">10</param>
+        <param name="SyncTable 2 Read Size 5">${num_taxels}</param>
         <param name="SyncTable 2 Write Address 1">230</param>
         <param name="SyncTable 2 Write Address 2">230</param>
@@ -312,5 +322,5 @@
         <param name="SyncTable 3 Read Size 3">6</param>
         <param name="SyncTable 3 Read Size 4">6</param>
-        <param name="SyncTable 3 Read Size 5">10</param>
+        <param name="SyncTable 3 Read Size 5">${num_taxels}</param>
         <param name="SyncTable 3 Write Address 1">230</param>
         <param name="SyncTable 3 Write Address 2">230</param>
@@ -332,5 +342,5 @@
         <param name="SyncTable 4 Read Size 3">6</param>
         <param name="SyncTable 4 Read Size 4">6</param>
-        <param name="SyncTable 4 Read Size 5">10</param>
+        <param name="SyncTable 4 Read Size 5">${num_taxels}</param>
         <param name="SyncTable 4 Write Address 1">230</param>
         <param name="SyncTable 4 Write Address 2">230</param>
@@ -352,5 +362,5 @@
         <param name="SyncTable 5 Read Size 3">6</param>
         <param name="SyncTable 5 Read Size 4">6</param>
-        <param name="SyncTable 5 Read Size 5">10</param>
+        <param name="SyncTable 5 Read Size 5">${num_taxels}</param>
         <param name="SyncTable 5 Write Address 1">230</param>
         <param name="SyncTable 5 Write Address 2">230</param>
@@ -892,5 +902,7 @@
         <state_interface name="Present Pressure 8"/>
         <state_interface name="Present Pressure 9"/>
-        <state_interface name="Present Pressure 10"/>
+        <xacro:if value="${int(num_taxels) == 10}">
+          <state_interface name="Present Pressure 10"/>
+        </xacro:if>
         <param name="type">virtual_sensor</param>
         <param name="ID">115</param>
@@ -952,5 +964,7 @@
         <state_interface name="Present Pressure 8"/>
         <state_interface name="Present Pressure 9"/>
-        <state_interface name="Present Pressure 10"/>
+        <xacro:if value="${int(num_taxels) == 10}">
+          <state_interface name="Present Pressure 10"/>
+        </xacro:if>
         <param name="type">virtual_sensor</param>
         <param name="ID">120</param>
@@ -1012,5 +1026,7 @@
         <state_interface name="Present Pressure 8"/>
         <state_interface name="Present Pressure 9"/>
-        <state_interface name="Present Pressure 10"/>
+        <xacro:if value="${int(num_taxels) == 10}">
+          <state_interface name="Present Pressure 10"/>
+        </xacro:if>
         <param name="type">virtual_sensor</param>
         <param name="ID">125</param>
@@ -1072,5 +1088,7 @@
         <state_interface name="Present Pressure 8"/>
         <state_interface name="Present Pressure 9"/>
-        <state_interface name="Present Pressure 10"/>
+        <xacro:if value="${int(num_taxels) == 10}">
+          <state_interface name="Present Pressure 10"/>
+        </xacro:if>
         <param name="type">virtual_sensor</param>
         <param name="ID">130</param>
@@ -1132,5 +1150,7 @@
         <state_interface name="Present Pressure 8"/>
         <state_interface name="Present Pressure 9"/>
-        <state_interface name="Present Pressure 10"/>
+        <xacro:if value="${int(num_taxels) == 10}">
+          <state_interface name="Present Pressure 10"/>
+        </xacro:if>
         <param name="type">virtual_sensor</param>
         <param name="ID">135</param>

File: robotis_hand_description/urdf/hx5_d20_rev1/hx5_d20_left.xacro (robot description, xacro)
@@ -1,4 +1,5 @@
 <?xml version="1.0"?>
 <robot name="hx5_d20_left" xmlns:xacro="http://www.ros.org/wiki/xacro">
+  <xacro:arg name="num_taxels" default="9" />
   <xacro:arg name="prefix" default="" />
   <xacro:arg name="use_sim" default="false" />
@@ -19,5 +20,6 @@
     name="HX5LeftSystem" prefix="$(arg prefix)" use_sim="$(arg use_sim)"
     use_mock_hardware="$(arg use_mock_hardware)"
-    mock_sensor_commands="$(arg mock_sensor_commands)"/>
+    mock_sensor_commands="$(arg mock_sensor_commands)"
+    num_taxels="$(arg num_taxels)"/>
   <gazebo>
     <plugin filename="gz_ros2_control-system" name="gz_ros2_control::GazeboSimROS2ControlPlugin">

File: robotis_hand_description/urdf/hx5_d20_rev1/hx5_d20_right.xacro (robot description, xacro)
@@ -1,4 +1,5 @@
 <?xml version="1.0"?>
 <robot name="hx5_d20_right" xmlns:xacro="http://www.ros.org/wiki/xacro">
+  <xacro:arg name="num_taxels" default="9" />
   <xacro:arg name="prefix" default="" />
   <xacro:arg name="use_sim" default="false" />
@@ -19,5 +20,6 @@
     name="HX5RightSystem" prefix="$(arg prefix)" use_sim="$(arg use_sim)"
     use_mock_hardware="$(arg use_mock_hardware)"
-    mock_sensor_commands="$(arg mock_sensor_commands)"/>
+    mock_sensor_commands="$(arg mock_sensor_commands)"
+    num_taxels="$(arg num_taxels)"/>
   <gazebo>
     <plugin filename="gz_ros2_control-system" name="gz_ros2_control::GazeboSimROS2ControlPlugin">

File: robotis_hand_description/urdf/hx5_d20_rev2/hx5_d20_left.xacro (robot description, xacro)
@@ -1,4 +1,5 @@
 <?xml version="1.0"?>
 <robot name="hx5_d20_left" xmlns:xacro="http://www.ros.org/wiki/xacro">
+  <xacro:arg name="num_taxels" default="9" />
   <xacro:arg name="prefix" default="" />
   <xacro:arg name="use_sim" default="false" />
@@ -19,5 +20,6 @@
     name="HX5LeftSystem" prefix="$(arg prefix)" use_sim="$(arg use_sim)"
     use_mock_hardware="$(arg use_mock_hardware)"
-    mock_sensor_commands="$(arg mock_sensor_commands)"/>
+    mock_sensor_commands="$(arg mock_sensor_commands)"
+    num_taxels="$(arg num_taxels)"/>
   <gazebo>
     <plugin filename="gz_ros2_control-system" name="gz_ros2_control::GazeboSimROS2ControlPlugin">

File: robotis_hand_description/urdf/hx5_d20_rev2/hx5_d20_right.xacro (robot description, xacro)
@@ -1,4 +1,5 @@
 <?xml version="1.0"?>
 <robot name="hx5_d20_right" xmlns:xacro="http://www.ros.org/wiki/xacro">
+  <xacro:arg name="num_taxels" default="9" />
   <xacro:arg name="prefix" default="" />
   <xacro:arg name="use_sim" default="false" />
@@ -19,5 +20,6 @@
     name="HX5RightSystem" prefix="$(arg prefix)" use_sim="$(arg use_sim)"
     use_mock_hardware="$(arg use_mock_hardware)"
-    mock_sensor_commands="$(arg mock_sensor_commands)"/>
+    mock_sensor_commands="$(arg mock_sensor_commands)"
+    num_taxels="$(arg num_taxels)"/>
   <gazebo>
     <plugin filename="gz_ros2_control-system" name="gz_ros2_control::GazeboSimROS2ControlPlugin">
