Commit message: Updated moveit config
Signed-off-by: Hyunwoo Nam <nhw@robotis.com>

File: robotis_hand_description/ros2_control/hx5_d20_rev2/hx5_d20_right.ros2_control.xacro (robot description, xacro)
@@ -389,11 +389,11 @@
         <param name="Startup Configuration">2</param>
         <param name="Operating Mode">5</param>
-        <param name="Drive Mode">13</param>
-        <param name="Bus Watchdog">100</param>
-        <param name="Profile Velocity">100</param>
-        <param name="Profile Acceleration">50</param>
-        <param name="Position P Gain">500</param>
-        <param name="Position D Gain">1000</param>
-        <param name="Homing Offset">1024</param>
+        <param name="Drive Mode">12</param>
+        <param name="Bus Watchdog">100</param>
+        <param name="Profile Velocity">100</param>
+        <param name="Profile Acceleration">50</param>
+        <param name="Position P Gain">500</param>
+        <param name="Position D Gain">1000</param>
+        <param name="Homing Offset">-1024</param>
         <param name="Indirect Address 1">126</param>
         <param name="Indirect Address 2">127</param>
@@ -413,5 +413,5 @@
         <param name="Startup Configuration">2</param>
         <param name="Operating Mode">5</param>
-        <param name="Drive Mode">13</param>
+        <param name="Drive Mode">12</param>
         <param name="Bus Watchdog">100</param>
         <param name="Profile Velocity">100</param>
@@ -436,5 +436,5 @@
         <param name="Startup Configuration">2</param>
         <param name="Operating Mode">5</param>
-        <param name="Drive Mode">13</param>
+        <param name="Drive Mode">12</param>
         <param name="Bus Watchdog">100</param>
         <param name="Profile Velocity">100</param>

File: robotis_hand_description/urdf/hx5_d20_rev2/hx5_d20_left.urdf.xacro (robot description, xacro)
@@ -191,5 +191,5 @@
          <parent link="${prefix}hx5_d20_left_base" />
          <child link="${prefix}finger_l_link5" />
-         <origin xyz="-0.0015 -0.03608 0.09575" rpy="0 0 0" />
+         <origin xyz="-0.0015 -0.03608 0.10275" rpy="0 0 0" />
          <axis xyz="1 0 0" />
          <limit velocity="4.8" effort="1000" lower="-0.6" upper="0.6" />
@@ -348,5 +348,5 @@
          <parent link="${prefix}hx5_d20_left_base" />
          <child link="${prefix}finger_l_link9" />
-         <origin xyz="-0.0015 -0.00908 0.10353" rpy="0 0 0" />
+         <origin xyz="-0.0015 -0.00908 0.11053" rpy="0 0 0" />
          <axis xyz="1 0 0" />
          <limit velocity="4.8" effort="1000" lower="-0.6" upper="0.6" />
@@ -505,5 +505,5 @@
          <parent link="${prefix}hx5_d20_left_base" />
          <child link="${prefix}finger_l_link13" />
-         <origin xyz="-0.0015 0.01792 0.09775" rpy="0 0 0" />
+         <origin xyz="-0.0015 0.01792 0.10475" rpy="0 0 0" />
          <axis xyz="1 0 0" />
          <limit velocity="4.8" effort="1000" lower="-0.6" upper="0.6" />
@@ -662,5 +662,5 @@
          <parent link="${prefix}hx5_d20_left_base" />
          <child link="${prefix}finger_l_link17" />
-         <origin xyz="-0.0015 0.04492 0.07875" rpy="0 0 0" />
+         <origin xyz="-0.0015 0.04492 0.08575" rpy="0 0 0" />
          <axis xyz="1 0 0" />
          <limit velocity="4.8" effort="1000" lower="-0.6" upper="0.6" />

File: robotis_hand_description/urdf/hx5_d20_rev2/hx5_d20_right.urdf.xacro (robot description, xacro)
@@ -191,5 +191,5 @@
          <parent link="${prefix}hx5_d20_right_base" />
          <child link="${prefix}finger_r_link5" />
-         <origin xyz="-0.0015 0.03608 0.09575" rpy="0 0 0" />
+         <origin xyz="-0.0015 0.03608 0.10275" rpy="0 0 0" />
          <axis xyz="1 0 0" />
          <limit velocity="4.8" effort="1000" lower="-0.6" upper="0.6" />
@@ -348,5 +348,5 @@
          <parent link="${prefix}hx5_d20_right_base" />
          <child link="${prefix}finger_r_link9" />
-         <origin xyz="-0.0015 0.00908 0.10353" rpy="0 0 0" />
+         <origin xyz="-0.0015 0.00908 0.11053" rpy="0 0 0" />
          <axis xyz="1 0 0" />
          <limit velocity="4.8" effort="1000" lower="-0.6" upper="0.6" />
@@ -505,5 +505,5 @@
          <parent link="${prefix}hx5_d20_right_base" />
          <child link="${prefix}finger_r_link13" />
-         <origin xyz="-0.0015 -0.01792 0.09775" rpy="0 0 0" />
+         <origin xyz="-0.0015 -0.01792 0.10475" rpy="0 0 0" />
          <axis xyz="1 0 0" />
          <limit velocity="4.8" effort="1000" lower="-0.6" upper="0.6" />
@@ -662,5 +662,5 @@
          <parent link="${prefix}hx5_d20_right_base" />
          <child link="${prefix}finger_r_link17" />
-         <origin xyz="-0.0015 -0.04492 0.07875" rpy="0 0 0" />
+         <origin xyz="-0.0015 -0.04492 0.08575" rpy="0 0 0" />
          <axis xyz="1 0 0" />
          <limit velocity="4.8" effort="1000" lower="-0.6" upper="0.6" />
