Commit message: Added pressure sensor
Signed-off-by: Hyunwoo Nam <nhw@robotis.com>

File: robotis_hand_description/ros2_control/hx5_d20_rev2/hx5_d20_right.ros2_control.xacro (robot description, xacro)
@@ -1,5 +1,5 @@
 <?xml version="1.0"?>
 <robot xmlns:xacro="http://www.ros.org/wiki/xacro">
-  <xacro:macro name="hx5_right_system" params="name prefix port_name:=^|/dev/ttyUSB0 use_sim:=^|false use_mock_hardware:=^|false mock_sensor_commands:=^|false">
+  <xacro:macro name="robotis_hand_system" params="name prefix port_name:=^|/dev/ttyUSB0 use_sim:=^|false use_mock_hardware:=^|false mock_sensor_commands:=^|false">
     <ros2_control name="${name}" type="system" is_async="true">
       <xacro:if value="$(arg use_sim)">
@@ -70,4 +70,5 @@
         <state_interface name="Present Pressure 8"/>
         <state_interface name="Present Pressure 9"/>
+        <state_interface name="Present Pressure 10"/>
       </sensor>
       <joint name="${prefix}finger_r_joint5">
@@ -109,4 +110,5 @@
         <state_interface name="Present Pressure 8"/>
         <state_interface name="Present Pressure 9"/>
+        <state_interface name="Present Pressure 10"/>
       </sensor>
       <joint name="${prefix}finger_r_joint9">
@@ -148,4 +150,5 @@
         <state_interface name="Present Pressure 8"/>
         <state_interface name="Present Pressure 9"/>
+        <state_interface name="Present Pressure 10"/>
       </sensor>
       <joint name="${prefix}finger_r_joint13">
@@ -187,4 +190,5 @@
         <state_interface name="Present Pressure 8"/>
         <state_interface name="Present Pressure 9"/>
+        <state_interface name="Present Pressure 10"/>
       </sensor>
       <joint name="${prefix}finger_r_joint17">
@@ -226,4 +230,5 @@
         <state_interface name="Present Pressure 8"/>
         <state_interface name="Present Pressure 9"/>
+        <state_interface name="Present Pressure 10"/>
       </sensor>
       <gpio name="hand_r_controller">
@@ -267,5 +272,5 @@
         <param name="SyncTable 1 Read Size 3">6</param>
         <param name="SyncTable 1 Read Size 4">6</param>
-        <param name="SyncTable 1 Read Size 5">9</param>
+        <param name="SyncTable 1 Read Size 5">10</param>
         <param name="SyncTable 1 Write Address 1">230</param>
         <param name="SyncTable 1 Write Address 2">230</param>
@@ -287,5 +292,5 @@
         <param name="SyncTable 2 Read Size 3">6</param>
         <param name="SyncTable 2 Read Size 4">6</param>
-        <param name="SyncTable 2 Read Size 5">9</param>
+        <param name="SyncTable 2 Read Size 5">10</param>
         <param name="SyncTable 2 Write Address 1">230</param>
         <param name="SyncTable 2 Write Address 2">230</param>
@@ -307,5 +312,5 @@
         <param name="SyncTable 3 Read Size 3">6</param>
         <param name="SyncTable 3 Read Size 4">6</param>
-        <param name="SyncTable 3 Read Size 5">9</param>
+        <param name="SyncTable 3 Read Size 5">10</param>
         <param name="SyncTable 3 Write Address 1">230</param>
         <param name="SyncTable 3 Write Address 2">230</param>
@@ -327,5 +332,5 @@
         <param name="SyncTable 4 Read Size 3">6</param>
         <param name="SyncTable 4 Read Size 4">6</param>
-        <param name="SyncTable 4 Read Size 5">9</param>
+        <param name="SyncTable 4 Read Size 5">10</param>
         <param name="SyncTable 4 Write Address 1">230</param>
         <param name="SyncTable 4 Write Address 2">230</param>
@@ -347,5 +352,5 @@
         <param name="SyncTable 5 Read Size 3">6</param>
         <param name="SyncTable 5 Read Size 4">6</param>
-        <param name="SyncTable 5 Read Size 5">9</param>
+        <param name="SyncTable 5 Read Size 5">10</param>
         <param name="SyncTable 5 Write Address 1">230</param>
         <param name="SyncTable 5 Write Address 2">230</param>
@@ -887,4 +892,5 @@
         <state_interface name="Present Pressure 8"/>
         <state_interface name="Present Pressure 9"/>
+        <state_interface name="Present Pressure 10"/>
         <param name="type">virtual_sensor</param>
         <param name="ID">115</param>
@@ -946,4 +952,5 @@
         <state_interface name="Present Pressure 8"/>
         <state_interface name="Present Pressure 9"/>
+        <state_interface name="Present Pressure 10"/>
         <param name="type">virtual_sensor</param>
         <param name="ID">120</param>
@@ -1005,4 +1012,5 @@
         <state_interface name="Present Pressure 8"/>
         <state_interface name="Present Pressure 9"/>
+        <state_interface name="Present Pressure 10"/>
         <param name="type">virtual_sensor</param>
         <param name="ID">125</param>
@@ -1064,4 +1072,5 @@
         <state_interface name="Present Pressure 8"/>
         <state_interface name="Present Pressure 9"/>
+        <state_interface name="Present Pressure 10"/>
         <param name="type">virtual_sensor</param>
         <param name="ID">130</param>
@@ -1123,4 +1132,5 @@
         <state_interface name="Present Pressure 8"/>
         <state_interface name="Present Pressure 9"/>
+        <state_interface name="Present Pressure 10"/>
         <param name="type">virtual_sensor</param>
         <param name="ID">135</param>

Commit message: Fixed typo
Signed-off-by: Hyunwoo Nam <nhw@robotis.com>

File: robotis_hand_description/ros2_control/hx5_d20_rev2/hx5_d20_right.ros2_control.xacro (robot description, xacro)
@@ -1,5 +1,5 @@
 <?xml version="1.0"?>
 <robot xmlns:xacro="http://www.ros.org/wiki/xacro">
-  <xacro:macro name="robotis_hand_system" params="name prefix port_name:=^|/dev/ttyUSB0 use_sim:=^|false use_mock_hardware:=^|false mock_sensor_commands:=^|false">
+  <xacro:macro name="hx5_right_system" params="name prefix port_name:=^|/dev/ttyUSB0 use_sim:=^|false use_mock_hardware:=^|false mock_sensor_commands:=^|false">
     <ros2_control name="${name}" type="system" is_async="true">
       <xacro:if value="$(arg use_sim)">
