Commit message: Update macro names
Signed-off-by: Hyunwoo Nam <nhw@robotis.com>

File: robotis_hand_description/gazebo/hx5_d20/hx5_d20_left.gazebo.xacro (robot description, xacro)
@@ -1,5 +1,5 @@
 <?xml version="1.0"?>
 <robot xmlns:xacro="http://ros.org/wiki/xacro">
-  <xacro:macro name="robotis_hand_gazebo" params="prefix">
+  <xacro:macro name="robotis_hand_left_gazebo" params="prefix">
   <xacro:macro name="SimpleTransmission" params="trans joint actuator">
     <transmission name="${trans}">

File: robotis_hand_description/gazebo/hx5_d20/hx5_d20_right.gazebo.xacro (robot description, xacro)
@@ -1,5 +1,5 @@
 <?xml version="1.0"?>
 <robot xmlns:xacro="http://ros.org/wiki/xacro">
-  <xacro:macro name="robotis_hand_gazebo" params="prefix">
+  <xacro:macro name="robotis_hand_right_gazebo" params="prefix">
   <xacro:macro name="SimpleTransmission" params="trans joint actuator">
     <transmission name="${trans}">

File: robotis_hand_description/ros2_control/hx5_d20_rev1/hx5_d20_left.ros2_control.xacro (robot description, xacro)
@@ -1,5 +1,5 @@
 <?xml version="1.0"?>
 <robot xmlns:xacro="http://www.ros.org/wiki/xacro">
-  <xacro:macro name="robotis_hand_system" params="name prefix port_name:=^|/dev/ttyUSB0 use_sim:=^|false use_mock_hardware:=^|false mock_sensor_commands:=^|false">
+  <xacro:macro name="hx5_left_system" params="name prefix port_name:=^|/dev/ttyUSB0 use_sim:=^|false use_mock_hardware:=^|false mock_sensor_commands:=^|false">
     <ros2_control name="${name}" type="system" is_async="true">
       <xacro:if value="$(arg use_sim)">

File: robotis_hand_description/ros2_control/hx5_d20_rev1/hx5_d20_right.ros2_control.xacro (robot description, xacro)
@@ -1,5 +1,5 @@
 <?xml version="1.0"?>
 <robot xmlns:xacro="http://www.ros.org/wiki/xacro">
-  <xacro:macro name="robotis_hand_system" params="name prefix port_name:=^|/dev/ttyUSB0 use_sim:=^|false use_mock_hardware:=^|false mock_sensor_commands:=^|false">
+  <xacro:macro name="hx5_right_system" params="name prefix port_name:=^|/dev/ttyUSB0 use_sim:=^|false use_mock_hardware:=^|false mock_sensor_commands:=^|false">
     <ros2_control name="${name}" type="system" is_async="true">
       <xacro:if value="$(arg use_sim)">

File: robotis_hand_description/ros2_control/hx5_d20_rev2/hx5_d20_left.ros2_control.xacro (robot description, xacro)
@@ -1,5 +1,5 @@
 <?xml version="1.0"?>
 <robot xmlns:xacro="http://www.ros.org/wiki/xacro">
-  <xacro:macro name="robotis_hand_system" params="name prefix port_name:=^|/dev/ttyUSB0 use_sim:=^|false use_mock_hardware:=^|false mock_sensor_commands:=^|false">
+  <xacro:macro name="hx5_left_system" params="name prefix port_name:=^|/dev/ttyUSB0 use_sim:=^|false use_mock_hardware:=^|false mock_sensor_commands:=^|false">
     <ros2_control name="${name}" type="system" is_async="true">
       <xacro:if value="$(arg use_sim)">

File: robotis_hand_description/ros2_control/hx5_d20_rev2/hx5_d20_right.ros2_control.xacro (robot description, xacro)
@@ -1,5 +1,5 @@
 <?xml version="1.0"?>
 <robot xmlns:xacro="http://www.ros.org/wiki/xacro">
-  <xacro:macro name="robotis_hand_system" params="name prefix port_name:=^|/dev/ttyUSB0 use_sim:=^|false use_mock_hardware:=^|false mock_sensor_commands:=^|false">
+  <xacro:macro name="hx5_right_system" params="name prefix port_name:=^|/dev/ttyUSB0 use_sim:=^|false use_mock_hardware:=^|false mock_sensor_commands:=^|false">
     <ros2_control name="${name}" type="system" is_async="true">
       <xacro:if value="$(arg use_sim)">

File: robotis_hand_description/urdf/hx5_d20_rev1/hx5_d20_left.xacro (robot description, xacro)
@@ -15,7 +15,7 @@
   </joint>
   <xacro:hx5_d20_left prefix="$(arg prefix)" />
-  <xacro:robotis_hand_gazebo prefix="$(arg prefix)" />
-  <xacro:robotis_hand_system
-    name="RobotisHandSystem" prefix="$(arg prefix)" use_sim="$(arg use_sim)"
+  <xacro:robotis_hand_left_gazebo prefix="$(arg prefix)" />
+  <xacro:hx5_left_system
+    name="HX5LeftSystem" prefix="$(arg prefix)" use_sim="$(arg use_sim)"
     use_mock_hardware="$(arg use_mock_hardware)"
     mock_sensor_commands="$(arg mock_sensor_commands)"/>

File: robotis_hand_description/urdf/hx5_d20_rev1/hx5_d20_right.xacro (robot description, xacro)
@@ -15,7 +15,7 @@
   </joint>
   <xacro:hx5_d20_right prefix="$(arg prefix)" />
-  <xacro:robotis_hand_gazebo prefix="$(arg prefix)" />
-  <xacro:robotis_hand_system
-    name="RobotisHandSystem" prefix="$(arg prefix)" use_sim="$(arg use_sim)"
+  <xacro:robotis_hand_right_gazebo prefix="$(arg prefix)" />
+  <xacro:hx5_right_system
+    name="HX5RightSystem" prefix="$(arg prefix)" use_sim="$(arg use_sim)"
     use_mock_hardware="$(arg use_mock_hardware)"
     mock_sensor_commands="$(arg mock_sensor_commands)"/>

File: robotis_hand_description/urdf/hx5_d20_rev2/hx5_d20_left.xacro (robot description, xacro)
@@ -15,7 +15,7 @@
   </joint>
   <xacro:hx5_d20_left prefix="$(arg prefix)" />
-  <xacro:robotis_hand_gazebo prefix="$(arg prefix)" />
-  <xacro:robotis_hand_system
-    name="RobotisHandSystem" prefix="$(arg prefix)" use_sim="$(arg use_sim)"
+  <xacro:robotis_hand_left_gazebo prefix="$(arg prefix)" />
+  <xacro:hx5_left_system
+    name="HX5LeftSystem" prefix="$(arg prefix)" use_sim="$(arg use_sim)"
     use_mock_hardware="$(arg use_mock_hardware)"
     mock_sensor_commands="$(arg mock_sensor_commands)"/>

File: robotis_hand_description/urdf/hx5_d20_rev2/hx5_d20_right.xacro (robot description, xacro)
@@ -15,7 +15,7 @@
   </joint>
   <xacro:hx5_d20_right prefix="$(arg prefix)" />
-  <xacro:robotis_hand_gazebo prefix="$(arg prefix)" />
-  <xacro:robotis_hand_system
-    name="RobotisHandSystem" prefix="$(arg prefix)" use_sim="$(arg use_sim)"
+  <xacro:robotis_hand_right_gazebo prefix="$(arg prefix)" />
+  <xacro:hx5_right_system
+    name="HX5RightSystem" prefix="$(arg prefix)" use_sim="$(arg use_sim)"
     use_mock_hardware="$(arg use_mock_hardware)"
     mock_sensor_commands="$(arg mock_sensor_commands)"/>
