Commit message: Updated URDF and CHANGELOG
Signed-off-by: Hyunwoo Nam <nhw@robotis.com>

File: robotis_hand_description/urdf/hx5_d20_rev2/hx5_d20_left.urdf.xacro (robot description, xacro)
@@ -164,9 +164,9 @@
          </collision>
          <inertial>
-            <origin xyz="6.6604979e-05 -1.6824458e-02 2.2398502e-04" />
-            <mass value="4.3875236e-02" />
-            <inertia ixx="1.1160744e-05" ixy="-8.5593479e-09" ixz="-1.7171147e-09"
-            iyy="2.8079428e-06" iyz="3.0446511e-07"
-            izz="1.1343106e-05" />
+            <origin xyz="-1.7938916e-05 -1.6839136e-02 2.3602399e-04" />
+            <mass value="4.3781048e-02" />
+            <inertia ixx="1.1225495e-05" ixy="1.5543842e-08" ixz="5.8360810e-10"
+            iyy="2.7956646e-06" iyz="3.1575945e-07"
+            izz="1.1392997e-05" />
          </inertial>
       </link>

Commit message: Add hx5_d20 keyboard teleop

File: robotis_hand_description/urdf/hx5_d20_rev2/hx5_d20_left.urdf.xacro (robot description, xacro)
@@ -71,5 +71,9 @@
          <origin xyz="0.039 0.0 0.0" rpy="0 0 0" />
          <axis xyz="0 0 1" />
+<<<<<<< HEAD
          <limit velocity="4.8" effort="1000" lower="0.0" upper="1.57" />
+=======
+         <limit velocity="4.8" effort="1000" lower="-0.5" upper="3.5" />
+>>>>>>> 4188d46 (Add hx5_d20 keyboard teleop)
          <dynamics damping="0.05" />
       </joint>
@@ -106,5 +110,5 @@
          <origin xyz="0.0 -0.028 0.0" rpy="0 0 0" />
          <axis xyz="1 0 0" />
-         <limit velocity="4.8" effort="1000" lower="-1.57" upper="0.0" />
+         <limit velocity="4.8" effort="1000" lower="-1.57" upper="0.5" />
          <dynamics damping="0.05" />
       </joint>
@@ -141,5 +145,5 @@
          <origin xyz="0.0 -0.0355 0.0" rpy="0 0 0" />
          <axis xyz="1 0 0" />
-         <limit velocity="4.8" effort="1000" lower="-1.57" upper="0.0" />
+         <limit velocity="4.8" effort="1000" lower="-1.57" upper="0.5" />
          <dynamics damping="0.05" />
       </joint>

File: robotis_hand_description/urdf/hx5_d20_rev2/hx5_d20_right.urdf.xacro (robot description, xacro)
@@ -71,5 +71,9 @@
          <origin xyz="0.039 0.0 0.0" rpy="0 0 0" />
          <axis xyz="0 0 1" />
+<<<<<<< HEAD
          <limit velocity="4.8" effort="1000" lower="-1.57" upper="0.0" />
+=======
+         <limit velocity="4.8" effort="1000" lower="-3.5" upper="0.5" />
+>>>>>>> 4188d46 (Add hx5_d20 keyboard teleop)
          <dynamics damping="0.05" />
       </joint>
@@ -106,5 +110,5 @@
          <origin xyz="0.0 0.028 0.0" rpy="0 0 0" />
          <axis xyz="1 0 0" />
-         <limit velocity="4.8" effort="1000" lower="0.0" upper="1.57" />
+         <limit velocity="4.8" effort="1000" lower="-0.5" upper="1.57" />
          <dynamics damping="0.05" />
       </joint>
@@ -141,5 +145,5 @@
          <origin xyz="0.0 0.0355 0.0" rpy="0 0 0" />
          <axis xyz="1 0 0" />
-         <limit velocity="4.8" effort="1000" lower="0.0" upper="1.57" />
+         <limit velocity="4.8" effort="1000" lower="-0.5" upper="1.57" />
          <dynamics damping="0.05" />
       </joint>

Commit message: Adjusted joint2 position limits to better emulate human range of motion
Signed-off-by: Hyunwoo Nam <nhw@robotis.com>

File: robotis_hand_description/urdf/hx5_d20_rev2/hx5_d20_left.urdf.xacro (robot description, xacro)
@@ -71,5 +71,5 @@
          <origin xyz="0.039 0.0 0.0" rpy="0 0 0" />
          <axis xyz="0 0 1" />
-         <limit velocity="4.8" effort="1000" lower="0.0" upper="3.14" />
+         <limit velocity="4.8" effort="1000" lower="0.0" upper="1.57" />
          <dynamics damping="0.05" />
       </joint>

File: robotis_hand_description/urdf/hx5_d20_rev2/hx5_d20_right.urdf.xacro (robot description, xacro)
@@ -71,5 +71,5 @@
          <origin xyz="0.039 0.0 0.0" rpy="0 0 0" />
          <axis xyz="0 0 1" />
-         <limit velocity="4.8" effort="1000" lower="-3.14" upper="0.0" />
+         <limit velocity="4.8" effort="1000" lower="-1.57" upper="0.0" />
          <dynamics damping="0.05" />
       </joint>

Commit message: Formatting package & setup.py

File: robotis_hand_description/urdf/hx5_d20_rev2/hx5_d20_left.urdf.xacro (robot description, xacro)
@@ -71,9 +71,5 @@
          <origin xyz="0.039 0.0 0.0" rpy="0 0 0" />
          <axis xyz="0 0 1" />
-<<<<<<< HEAD
-         <limit velocity="4.8" effort="1000" lower="0.0" upper="1.57" />
-=======
-         <limit velocity="4.8" effort="1000" lower="-0.5" upper="3.5" />
->>>>>>> 4188d46 (Add hx5_d20 keyboard teleop)
+         <limit velocity="4.8" effort="1000" lower="0.0" upper="2.57" />
          <dynamics damping="0.05" />
       </joint>

File: robotis_hand_description/urdf/hx5_d20_rev2/hx5_d20_right.urdf.xacro (robot description, xacro)
@@ -71,9 +71,5 @@
          <origin xyz="0.039 0.0 0.0" rpy="0 0 0" />
          <axis xyz="0 0 1" />
-<<<<<<< HEAD
-         <limit velocity="4.8" effort="1000" lower="-1.57" upper="0.0" />
-=======
-         <limit velocity="4.8" effort="1000" lower="-3.5" upper="0.5" />
->>>>>>> 4188d46 (Add hx5_d20 keyboard teleop)
+         <limit velocity="4.8" effort="1000" lower="-2.57" upper="0.0" />
          <dynamics damping="0.05" />
       </joint>

Commit message: Restoring urdf

File: robotis_hand_description/urdf/hx5_d20_rev2/hx5_d20_left.urdf.xacro (robot description, xacro)
@@ -71,5 +71,5 @@
          <origin xyz="0.039 0.0 0.0" rpy="0 0 0" />
          <axis xyz="0 0 1" />
-         <limit velocity="4.8" effort="1000" lower="0.0" upper="2.57" />
+         <limit velocity="4.8" effort="1000" lower="0.0" upper="1.57" />
          <dynamics damping="0.05" />
       </joint>
@@ -106,5 +106,5 @@
          <origin xyz="0.0 -0.028 0.0" rpy="0 0 0" />
          <axis xyz="1 0 0" />
-         <limit velocity="4.8" effort="1000" lower="-1.57" upper="0.5" />
+         <limit velocity="4.8" effort="1000" lower="-1.57" upper="0.0" />
          <dynamics damping="0.05" />
       </joint>
@@ -141,5 +141,5 @@
          <origin xyz="0.0 -0.0355 0.0" rpy="0 0 0" />
          <axis xyz="1 0 0" />
-         <limit velocity="4.8" effort="1000" lower="-1.57" upper="0.5" />
+         <limit velocity="4.8" effort="1000" lower="-1.57" upper="0.0" />
          <dynamics damping="0.05" />
       </joint>

File: robotis_hand_description/urdf/hx5_d20_rev2/hx5_d20_right.urdf.xacro (robot description, xacro)
@@ -71,5 +71,5 @@
          <origin xyz="0.039 0.0 0.0" rpy="0 0 0" />
          <axis xyz="0 0 1" />
-         <limit velocity="4.8" effort="1000" lower="-2.57" upper="0.0" />
+         <limit velocity="4.8" effort="1000" lower="-1.57" upper="0.0" />
          <dynamics damping="0.05" />
       </joint>
@@ -106,5 +106,5 @@
          <origin xyz="0.0 0.028 0.0" rpy="0 0 0" />
          <axis xyz="1 0 0" />
-         <limit velocity="4.8" effort="1000" lower="-0.5" upper="1.57" />
+         <limit velocity="4.8" effort="1000" lower="0.0" upper="1.57" />
          <dynamics damping="0.05" />
       </joint>
@@ -141,5 +141,5 @@
          <origin xyz="0.0 0.0355 0.0" rpy="0 0 0" />
          <axis xyz="1 0 0" />
-         <limit velocity="4.8" effort="1000" lower="-0.5" upper="1.57" />
+         <limit velocity="4.8" effort="1000" lower="0.0" upper="1.57" />
          <dynamics damping="0.05" />
       </joint>
