Commit message: Fixed typo
Signed-off-by: Hyunwoo Nam <nhw@robotis.com>

File: robotis_hand_description/urdf/hx5_d20_rev1/hx5_d20_left.urdf.xacro (robot description, xacro)
@@ -2,5 +2,5 @@
 <robot xmlns:xacro="http://www.ros.org/wiki/xacro">
    <xacro:macro name="hx5_d20_left" params="prefix">
-      <xacro:property name="meshes_file_direction" value="package://robotis_hand_description/meshes/hx5_d20_rev1/hx5_d20_left/" />
+      <xacro:property name="meshes_file_direction" value="package://robotis_hand_description/meshes/hx5_d20_rev1/hx5_d20_left" />
       <link name="${prefix}hx5_d20_left_base">
          <visual>

File: robotis_hand_description/urdf/hx5_d20_rev1/hx5_d20_right.urdf.xacro (robot description, xacro)
@@ -2,5 +2,5 @@
 <robot xmlns:xacro="http://www.ros.org/wiki/xacro">
    <xacro:macro name="hx5_d20_right" params="prefix">
-      <xacro:property name="meshes_file_direction" value="package://robotis_hand_description/meshes/hx5_d20_rev1/hx5_d20_right/" />
+      <xacro:property name="meshes_file_direction" value="package://robotis_hand_description/meshes/hx5_d20_rev1/hx5_d20_right" />
       <link name="${prefix}hx5_d20_right_base">
          <visual>

File: robotis_hand_description/urdf/hx5_d20_rev2/hx5_d20_left.urdf.xacro (robot description, xacro)
@@ -2,5 +2,5 @@
 <robot xmlns:xacro="http://www.ros.org/wiki/xacro">
    <xacro:macro name="hx5_d20_left" params="prefix">
-      <xacro:property name="meshes_file_direction" value="package://robotis_hand_description/meshes/hx5_d20_rev2/hx5_d20_left/" />
+      <xacro:property name="meshes_file_direction" value="package://robotis_hand_description/meshes/hx5_d20_rev2/hx5_d20_left" />
       <link name="${prefix}hx5_d20_left_base">
          <visual>

File: robotis_hand_description/urdf/hx5_d20_rev2/hx5_d20_right.urdf.xacro (robot description, xacro)
@@ -2,5 +2,5 @@
 <robot xmlns:xacro="http://www.ros.org/wiki/xacro">
    <xacro:macro name="hx5_d20_right" params="prefix">
-      <xacro:property name="meshes_file_direction" value="package://robotis_hand_description/meshes/hx5_d20_rev2/hx5_d20_right/" />
+      <xacro:property name="meshes_file_direction" value="package://robotis_hand_description/meshes/hx5_d20_rev2/hx5_d20_right" />
       <link name="${prefix}hx5_d20_right_base">
          <visual>
